Commit message: Processed and robot list generated for next step

File: zoo/processed/ABB/IRB2400/irb2400.urdf (robot description, URDF)
Before this commit: robot abb_irb4400l_30_243, 9 links, 8 joints
Links:
- added link link_lever_a; collision mesh filename=package://abb_irb2400_support/meshes/irb2400_common/collisi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; visual mesh filename=package://abb_irb2400_support/meshes/irb2400_common/visual/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
- added link link_lever_b; collision mesh filename=package://abb_irb2400_support/meshes/irb2400_common/collisi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; visual mesh filename=package://abb_irb2400_support/meshes/irb2400_common/visual/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
- link base_link: geometry collision mesh filename=package://abb_irb2400_support/meshes/irb2400_common/collisi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; visual mesh filename=package://abb_irb2400_support/meshes/irb2400_common/visual/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
- link link_1: geometry collision mesh filename=package://abb_irb2400_support/meshes/irb2400_common/collisi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; visual mesh filename=package://abb_irb2400_support/meshes/irb2400_common/visual/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
- link link_2: geometry collision mesh filename=package://abb_irb2400_support/meshes/irb2400_common/collisi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; visual mesh filename=package://abb_irb2400_support/meshes/irb2400_common/visual/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
- link link_3: geometry collision mesh filename=package://abb_irb2400_support/meshes/irb2400_common/collisi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; visual mesh filename=package://abb_irb2400_support/meshes/irb2400_common/visual/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
- link link_4: geometry collision mesh filename=package://abb_irb2400_support/meshes/irb2400_common/collisi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; visual mesh filename=package://abb_irb2400_support/meshes/irb2400_common/visual/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
- link link_5: geometry collision mesh filename=package://abb_irb2400_support/meshes/irb2400_common/collisi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; visual mesh filename=package://abb_irb2400_support/meshes/irb2400_common/visual/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
- link link_6: geometry collision mesh filename=package://abb_irb2400_support/meshes/irb2400_common/collisi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; visual mesh filename=package://abb_irb2400_support/meshes/irb2400_common/visual/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
Joints:
- added joint joint_lever_a: type continuous, parent link_2, child link_lever_a, origin xyz=0 0 0 rpy=0 0 0, axis 0 1 0, mimic joint=joint_3 multiplier=1.0
- added joint joint_lever_b: type continuous, parent link_3, child link_lever_b, origin xyz=-0.18 0 0 rpy=0 0 0, axis 0 1 0, mimic joint=joint_3 multiplier=-1.0
- joint joint_1: limit lower=-2.87979 upper=2.87979 effort=0 velocity=2.618 -> lower=-3.1416 upper=3.1416 effort=0 velocity=2.618
- joint joint_2: limit lower=-1.2217 upper=1.658 effort=0 velocity=2.0944 -> lower=-1.7453 upper=1.9199 effort=0 velocity=2.618; origin xyz=0.2 0 0.68 rpy=0 0 0 -> xyz=0.1 0 0.615 rpy=0 0 0
- joint joint_3: limit lower=-1.0472 upper=1.1345 effort=0 velocity=2.0944 -> lower=-1.0472 upper=1.1345 effort=0 velocity=2.618; origin xyz=0 0 0.89 rpy=0 0 0 -> xyz=0 0 0.705 rpy=0 0 0
- joint joint_4: limit lower=-3.49 upper=3.49 effort=0 velocity=3.927 -> lower=-3.49 upper=3.49 effort=0 velocity=6.2832; origin xyz=1.38 0 0.15 rpy=0 0 0 -> xyz=0 0 0.135 rpy=0 0 0
- joint joint_5: limit lower=-2.0944 upper=2.0944 effort=0 velocity=4.3633 -> lower=-2.0944 upper=2.0944 effort=0 velocity=6.2832; origin xyz=0 0 0 rpy=0 0 0 -> xyz=0.755 0 0 rpy=0 0 0
- joint joint_6: limit lower=-6.9813 upper=6.9813 effort=0 velocity=5.7596 -> lower=-6.9813 upper=6.9813 effort=0 velocity=7.854
- joint joint_6-tool0: origin xyz=0.14 0 0 rpy=0 0 0 -> xyz=0.085 0 0 rpy=0 1.57079632679 0

File: zoo/processed/ABB/IRB4400/irb4400.urdf (robot description, URDF)
Before this commit: robot abb_irb2400_12_155, 11 links, 10 joints
Links:
- removed link link_lever_a
- removed link link_lever_b
- link base_link: geometry collision mesh filename=package://abb_irb4400_support/meshes/irb4400l_30_243/collis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; visual mesh filename=package://abb_irb4400_support/meshes/irb4400l_30_243/visual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
- link link_1: geometry collision mesh filename=package://abb_irb4400_support/meshes/irb4400l_30_243/collis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; visual mesh filename=package://abb_irb4400_support/meshes/irb4400l_30_243/visual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
- link link_2: geometry collision mesh filename=package://abb_irb4400_support/meshes/irb4400l_30_243/collis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; visual mesh filename=package://abb_irb4400_support/meshes/irb4400l_30_243/visual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
- link link_3: geometry collision mesh filename=package://abb_irb4400_support/meshes/irb4400l_30_243/collis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; visual mesh filename=package://abb_irb4400_support/meshes/irb4400l_30_243/visual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
- link link_4: geometry collision mesh filename=package://abb_irb4400_support/meshes/irb4400l_30_243/collis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; visual mesh filename=package://abb_irb4400_support/meshes/irb4400l_30_243/visual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
- link link_5: geometry collision mesh filename=package://abb_irb4400_support/meshes/irb4400l_30_243/collis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; visual mesh filename=package://abb_irb4400_support/meshes/irb4400l_30_243/visual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
- link link_6: geometry collision mesh filename=package://abb_irb4400_support/meshes/irb4400l_30_243/collis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; visual mesh filename=package://abb_irb4400_support/meshes/irb4400l_30_243/visual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
Joints:
- removed joint joint_lever_a
- removed joint joint_lever_b
- joint joint_1: limit lower=-3.1416 upper=3.1416 effort=0 velocity=2.618 -> lower=-2.87979 upper=2.87979 effort=0 velocity=2.618
- joint joint_2: limit lower=-1.7453 upper=1.9199 effort=0 velocity=2.618 -> lower=-1.2217 upper=1.658 effort=0 velocity=2.0944; origin xyz=0.1 0 0.615 rpy=0 0 0 -> xyz=0.2 0 0.68 rpy=0 0 0
- joint joint_3: limit lower=-1.0472 upper=1.1345 effort=0 velocity=2.618 -> lower=-1.0472 upper=1.1345 effort=0 velocity=2.0944; origin xyz=0 0 0.705 rpy=0 0 0 -> xyz=0 0 0.89 rpy=0 0 0
- joint joint_4: limit lower=-3.49 upper=3.49 effort=0 velocity=6.2832 -> lower=-3.49 upper=3.49 effort=0 velocity=3.927; origin xyz=0 0 0.135 rpy=0 0 0 -> xyz=1.38 0 0.15 rpy=0 0 0
- joint joint_5: limit lower=-2.0944 upper=2.0944 effort=0 velocity=6.2832 -> lower=-2.0944 upper=2.0944 effort=0 velocity=4.3633; origin xyz=0.755 0 0 rpy=0 0 0 -> xyz=0 0 0 rpy=0 0 0
- joint joint_6: limit lower=-6.9813 upper=6.9813 effort=0 velocity=7.854 -> lower=-6.9813 upper=6.9813 effort=0 velocity=5.7596
- joint joint_6-tool0: origin xyz=0.085 0 0 rpy=0 1.57079632679 0 -> xyz=0.14 0 0 rpy=0 0 0

Commit message: Added franka robots to ABB dir for testing

File: zoo/processed/ABB/IRB2400/irb2400.urdf (robot description, URDF)
Before this commit: robot abb_irb2400_12_155, 11 links, 10 joints
Links:
- link base_link: geometry collision mesh filename=package://meshes/irb2400_common/collision/base_link.dae; visual mesh filename=package://meshes/irb2400_common/visual/base_link.dae
- link link_1: geometry collision mesh filename=package://meshes/irb2400_common/collision/link_1.dae; visual mesh filename=package://meshes/irb2400_common/visual/link_1.dae
- link link_2: geometry collision mesh filename=package://meshes/irb2400_common/collision/link_2.dae; visual mesh filename=package://meshes/irb2400_common/visual/link_2.dae
- link link_3: geometry collision mesh filename=package://meshes/irb2400_common/collision/link_3.dae; visual mesh filename=package://meshes/irb2400_common/visual/link_3.dae
- link link_4: geometry collision mesh filename=package://meshes/irb2400_common/collision/link_4.dae; visual mesh filename=package://meshes/irb2400_common/visual/link_4.dae
- link link_5: geometry collision mesh filename=package://meshes/irb2400_common/collision/link_5.dae; visual mesh filename=package://meshes/irb2400_common/visual/link_5.dae
- link link_6: geometry collision mesh filename=package://meshes/irb2400_common/collision/link_6.dae; visual mesh filename=package://meshes/irb2400_common/visual/link_6.dae
- link link_lever_a: geometry collision mesh filename=package://meshes/irb2400_common/collision/link_lever_a.dae; visual mesh filename=package://meshes/irb2400_common/visual/link_lever_a.dae
- link link_lever_b: geometry collision mesh filename=package://meshes/irb2400_common/collision/link_lever_b.dae; visual mesh filename=package://meshes/irb2400_common/visual/link_lever_b.dae

File: zoo/processed/ABB/IRB4400/irb4400.urdf (robot description, URDF)
Before this commit: robot abb_irb4400l_30_243, 9 links, 8 joints
Links:
- link base_link: geometry collision mesh filename=package://meshes/irb4400l_30_243/collision/base_link.dae; visual mesh filename=package://meshes/irb4400l_30_243/visual/base_link.dae
- link link_1: geometry collision mesh filename=package://meshes/irb4400l_30_243/collision/link_1.dae; visual mesh filename=package://meshes/irb4400l_30_243/visual/link_1.dae
- link link_2: geometry collision mesh filename=package://meshes/irb4400l_30_243/collision/link_2.dae; visual mesh filename=package://meshes/irb4400l_30_243/visual/link_2.dae
- link link_3: geometry collision mesh filename=package://meshes/irb4400l_30_243/collision/link_3.dae; visual mesh filename=package://meshes/irb4400l_30_243/visual/link_3.dae
- link link_4: geometry collision mesh filename=package://meshes/irb4400l_30_243/collision/link_4.dae; visual mesh filename=package://meshes/irb4400l_30_243/visual/link_4.dae
- link link_5: geometry collision mesh filename=package://meshes/irb4400l_30_243/collision/link_5.dae; visual mesh filename=package://meshes/irb4400l_30_243/visual/link_5.dae
- link link_6: geometry collision mesh filename=package://meshes/irb4400l_30_243/collision/link_6.dae; visual mesh filename=package://meshes/irb4400l_30_243/visual/link_6.dae

File: zoo/processed/ABB/IRB5400/irb5400.urdf (robot description, URDF)
Before this commit: robot abb_irb5400, 10 links, 9 joints
Links:
- link base_link: geometry collision mesh filename=package://meshes/irb5400/collision/base_link.stl; visual mesh filename=package://meshes/irb5400/visual/base_link.dae
- link link_1: geometry collision mesh filename=package://meshes/irb5400/collision/link_1.stl; visual mesh filename=package://meshes/irb5400/visual/link_1.dae
- link link_2: geometry collision mesh filename=package://meshes/irb5400/collision/link_2.stl; visual mesh filename=package://meshes/irb5400/visual/link_2.dae
- link link_3: geometry collision mesh filename=package://meshes/irb5400/collision/link_3.stl; visual mesh filename=package://meshes/irb5400/visual/link_3.dae
- link link_4: geometry collision mesh filename=package://meshes/irb5400/collision/link_4.stl; visual mesh filename=package://meshes/irb5400/visual/link_4.dae
- link link_5: geometry collision mesh filename=package://meshes/irb5400/collision/link_5.stl; visual mesh filename=package://meshes/irb5400/visual/link_5.dae
- link link_5b: geometry collision mesh filename=package://meshes/irb5400/collision/link_5b.stl; visual mesh filename=package://meshes/irb5400/visual/link_5b.dae
- link link_6: geometry collision mesh filename=package://meshes/irb5400/collision/link_6.stl; visual mesh filename=package://meshes/irb5400/visual/link_6.dae
Joints:
- joint joint5b: origin xyz=.106246 0 0.074394 rpy=0 -1.2217 0 -> xyz=0.106246 0 0.074394 rpy=0 -1.2217 0

File: zoo/processed/ABB/IRB6600/irb6600.urdf (robot description, URDF)
Before this commit: robot abb_irb6600_225_255, 11 links, 10 joints
Links:
- link base_link: geometry collision mesh filename=package://meshes/irb6600_225_255/collision/base_link.dae; visual mesh filename=package://meshes/irb6600_225_255/visual/base_link.dae
- link link_1: geometry collision mesh filename=package://meshes/irb6600_225_255/collision/link_1.dae; visual mesh filename=package://meshes/irb6600_225_255/visual/link_1.dae
- link link_2: geometry collision mesh filename=package://meshes/irb6600_225_255/collision/link_2.dae; visual mesh filename=package://meshes/irb6600_225_255/visual/link_2.dae
- link link_3: geometry collision mesh filename=package://meshes/irb6600_225_255/collision/link_3.dae; visual mesh filename=package://meshes/irb6600_225_255/visual/link_3.dae
- link link_4: geometry collision mesh filename=package://meshes/irb6600_225_255/collision/link_4.dae; visual mesh filename=package://meshes/irb6600_225_255/visual/link_4.dae
- link link_5: geometry collision mesh filename=package://meshes/irb6600_225_255/collision/link_5.dae; visual mesh filename=package://meshes/irb6600_225_255/visual/link_5.dae
- link link_6: geometry collision mesh filename=package://meshes/irb6600_225_255/collision/link_6.dae; visual mesh filename=package://meshes/irb6600_225_255/visual/link_6.dae
- link link_cylinder: geometry collision mesh filename=package://meshes/irb6600_225_255/collision/link_cylinder.dae; visual mesh filename=package://meshes/irb6600_225_255/visual/link_cylinder.dae
- link link_piston: geometry collision mesh filename=package://meshes/irb6600_225_255/collision/link_piston.dae; visual mesh filename=package://meshes/irb6600_225_255/visual/link_piston.dae

File: zoo/processed/ABB/IRB6640/irb6640.urdf (robot description, URDF)
Before this commit: robot abb_irb6640_185_280, 11 links, 10 joints
Links:
- link base_link: geometry collision mesh filename=package://meshes/irb6640_185_280/collision/base_link.dae; visual mesh filename=package://meshes/irb6640_185_280/visual/base_link.dae
- link link_1: geometry collision mesh filename=package://meshes/irb6640_185_280/collision/link_1.dae; visual mesh filename=package://meshes/irb6640_185_280/visual/link_1.dae
- link link_2: geometry collision mesh filename=package://meshes/irb6640_185_280/collision/link_2.dae; visual mesh filename=package://meshes/irb6640_185_280/visual/link_2.dae
- link link_3: geometry collision mesh filename=package://meshes/irb6640_185_280/collision/link_3.dae; visual mesh filename=package://meshes/irb6640_185_280/visual/link_3.dae
- link link_4: geometry collision mesh filename=package://meshes/irb6640_185_280/collision/link_4.dae; visual mesh filename=package://meshes/irb6640_185_280/visual/link_4.dae
- link link_5: geometry collision mesh filename=package://meshes/irb6640_185_280/collision/link_5.dae; visual mesh filename=package://meshes/irb6640_185_280/visual/link_5.dae
- link link_6: geometry collision mesh filename=package://meshes/irb6640_185_280/collision/link_6.dae; visual mesh filename=package://meshes/irb6640_185_280/visual/link_6.dae
- link link_cylinder: geometry collision mesh filename=package://meshes/irb6640_185_280/collision/cylinder_link.dae; visual mesh filename=package://meshes/irb6640_185_280/visual/cylinder_link.dae
- link link_piston: geometry collision mesh filename=package://meshes/irb6640_185_280/collision/piston_link.dae; visual mesh filename=package://meshes/irb6640_185_280/visual/piston_link.dae
