Commit message: IRB5400 xacro fix

File: zoo/processed/ABB/IRB5400/xacro/irb5400_macro.xacro (robot description, xacro)
@@ -159,5 +159,5 @@
         <parent link="${prefix}link_5"/>
         <child link="${prefix}link_5b"/>
-        <origin xyz=".106246 0 0.074394" rpy="0 -1.2217 0"/>
+        <origin xyz="0.106246 0 0.074394" rpy="0 -1.2217 0"/>
         <axis xyz="1 0 0"/>
         <limit lower="-6.0" upper="6.0" effort="100" velocity="6.1086"/>

Commit message: Removed ROS to tool transform

File: zoo/processed/ABB/IRB5400/xacro/irb5400_macro.xacro (robot description, xacro)
@@ -177,11 +177,4 @@
     </joint>
     <!-- end of joint list -->
-    <!-- ROS base_link to ABB World Coordinates transform -->
-    <link name="${prefix}base" />
-    <joint name="${prefix}base_link-base" type="fixed">
-        <origin xyz="0 0 0" rpy="0 0 0"/>
-        <parent link="${prefix}base_link"/>
-        <child link="${prefix}base"/>
-    </joint>
 </xacro:macro>
 </robot>
