Commit message: PR2 update

File: zoo/processed/Clearpath/PR2/xacro/gripper_v0/gripper.urdf.xacro (robot description, xacro)
@@ -188,5 +188,5 @@
     <joint name="${side}_gripper_led_joint" type="fixed">
       <!--  Need to check if we need a positive or negative Z term -->
-      <origin xyz="0.0513 0.0 0.0244"/>
+      <origin xyz="0.0513 0.0 .0244"/>
       <parent link="${side}_gripper_palm_link"/>
       <child link="${side}_gripper_led_frame"/>

File: zoo/processed/Clearpath/PR2/xacro/pr2.urdf.xacro (robot description, xacro)
@@ -109,5 +109,5 @@
                           frame_id="l_forearm_cam_optical_frame" hack_baseline="0"
                           image_width="640" image_height="480">
-    <origin xyz="0.135 0 0.044" rpy="${-M_PI/2} ${-32.25*M_PI/180} 0" />
+    <origin xyz=".135 0 .044" rpy="${-M_PI/2} ${-32.25*M_PI/180} 0" />
   </xacro:wge100_camera_v0>
   <xacro:wge100_camera_v0 name="r_forearm_cam" image_format="R8G8B8" camera_name="r_forearm_cam" image_topic_name="image_raw"
@@ -116,5 +116,5 @@
                           frame_id="r_forearm_cam_optical_frame" hack_baseline="0"
                           image_width="640" image_height="480">
-    <origin xyz="0.135 0 0.044" rpy="${M_PI/2} ${-32.25*M_PI/180} 0" />
+    <origin xyz=".135 0 .044" rpy="${M_PI/2} ${-32.25*M_PI/180} 0" />
   </xacro:wge100_camera_v0>
   <!-- Kinect models -->

File: zoo/processed/Clearpath/PR2/xacro/pr2_no_kinect.urdf.xacro (robot description, xacro)
@@ -109,5 +109,5 @@
                           frame_id="l_forearm_cam_optical_frame" hack_baseline="0"
                           image_width="640" image_height="480">
-    <origin xyz="0.135 0 0.044" rpy="${-M_PI/2} ${-32.25*M_PI/180} 0" />
+    <origin xyz=".135 0 .044" rpy="${-M_PI/2} ${-32.25*M_PI/180} 0" />
   </xacro:wge100_camera_v0>
   <xacro:wge100_camera_v0 name="r_forearm_cam" image_format="R8G8B8" camera_name="r_forearm_cam" image_topic_name="image_raw"
@@ -116,5 +116,5 @@
                           frame_id="r_forearm_cam_optical_frame" hack_baseline="0"
                           image_width="640" image_height="480">
-    <origin xyz="0.135 0 0.044" rpy="${M_PI/2} ${-32.25*M_PI/180} 0" />
+    <origin xyz=".135 0 .044" rpy="${M_PI/2} ${-32.25*M_PI/180} 0" />
   </xacro:wge100_camera_v0>
 </robot>

File: zoo/processed/Clearpath/PR2/xacro/pr2_se.urdf.xacro (robot description, xacro)
@@ -122,5 +122,5 @@
                           frame_id="r_forearm_cam_optical_frame" hack_baseline="0"
                           image_width="640" image_height="480">
-    <origin xyz="0.135 0 0.044" rpy="${M_PI/2} ${-32.25*M_PI/180} 0" />
+    <origin xyz=".135 0 .044" rpy="${M_PI/2} ${-32.25*M_PI/180} 0" />
   </xacro:wge100_camera_v0>
   <!-- PR2 SE does not have a left arm, so no left forearm camera :)
@@ -130,5 +130,5 @@
                           frame_id="l_forearm_cam_optical_frame" hack_baseline="0"
                           image_width="640" image_height="480">
-    <origin xyz="0.135 0 0.044" rpy="${-M_PI/2} ${-32.25*M_PI/180} 0" />
+    <origin xyz=".135 0 .044" rpy="${-M_PI/2} ${-32.25*M_PI/180} 0" />
   </xacro:wge100_camera_v0>
   -->
