Commit message: Addition of bow tags

File: zoo/processed/ABB/IRB2400/xacro/irb2400_12_155_macro.xacro (robot description, xacro)
@@ -147,5 +147,7 @@
       </collision>
     </link>
-    <link name="${prefix}tool0"/>
+    <link name="${prefix}tool0">
+        <bow name="arm" functions="goto point"/>
+    </link>
     <!-- end of link list -->
     <!-- joint list -->

File: zoo/processed/ABB/IRB4400/xacro/irb4400l_30_243_macro.xacro (robot description, xacro)
@@ -115,5 +115,7 @@
       </collision>
     </link>
-    <link name="${prefix}tool0"/>
+    <link name="${prefix}tool0">
+        <bow name="arm" functions="goto point"/>
+    </link>
     <!-- end of link list -->
     <!-- joint list -->

File: zoo/processed/ABB/IRB5400/xacro/irb5400_macro.xacro (robot description, xacro)
@@ -116,5 +116,7 @@
         </collision>
     </link>
-    <link name="${prefix}tool0"/>
+    <link name="${prefix}tool0">
+        <bow name="arm" functions="goto point"/>
+    </link>
     <!-- end of link list -->
     <!-- joint list -->

File: zoo/processed/ABB/IRB6600/xacro/irb6600_225_255_macro.xacro (robot description, xacro)
@@ -136,4 +136,5 @@
         <xacro:material_abb_yellow />
       </collision>
+      <bow name="arm" functions="goto point"/>
     </link>
     <!-- end of link list -->

File: zoo/processed/ABB/IRB6640/xacro/irb6640_185_280_macro.xacro (robot description, xacro)
@@ -123,4 +123,5 @@
         <material name="yellow"/>
       </visual>
+      <bow name="arm" functions="goto point"/>
     </link>
     <!-- end of link list -->

Commit message: ABB xacro update with BOW tags

File: zoo/processed/ABB/IRB2400/xacro/irb2400_12_155_macro.xacro (robot description, xacro)
@@ -148,5 +148,5 @@
     </link>
     <link name="${prefix}tool0">
-        <bow name="arm" functions="goto point"/>
+        <bow tags="effector"/>
     </link>
     <!-- end of link list -->
@@ -214,11 +214,4 @@
     </joint>
     <!-- end of joint list -->
-    <!-- ROS base_link to ABB World Coordinates transform -->
-    <link name="${prefix}base" />
-    <joint name="${prefix}base_link-base" type="fixed">
-      <origin xyz="0 0 0" rpy="0 0 0"/>
-      <parent link="${prefix}base_link"/>
-      <child link="${prefix}base"/>
-    </joint>
   </xacro:macro>
 </robot>

File: zoo/processed/ABB/IRB4400/xacro/irb4400l_30_243_macro.xacro (robot description, xacro)
@@ -116,5 +116,5 @@
     </link>
     <link name="${prefix}tool0">
-        <bow name="arm" functions="goto point"/>
+        <bow tags="effector"/>
     </link>
     <!-- end of link list -->
@@ -168,11 +168,4 @@
     </joint>
     <!-- end of joint list -->
-    <!-- ROS base_link to ABB World Coordinates transform -->
-    <link name="${prefix}base" />
-    <joint name="${prefix}base_link-base" type="fixed">
-      <origin xyz="0 0 0" rpy="0 0 0"/>
-      <parent link="${prefix}base_link"/>
-      <child link="${prefix}base"/>
-    </joint>
   </xacro:macro>
 </robot>

File: zoo/processed/ABB/IRB6600/xacro/irb6600_225_255_macro.xacro (robot description, xacro)
@@ -109,5 +109,7 @@
       </collision>
     </link>
-    <link name="${prefix}tool0" />
+    <link name="${prefix}tool0">
+        <bow tags="effector"/>
+    </link>
     <!--Cylinder and piston -->
     <link name="${prefix}link_cylinder">
@@ -136,5 +138,4 @@
         <xacro:material_abb_yellow />
       </collision>
-      <bow name="arm" functions="goto point"/>
     </link>
     <!-- end of link list -->
@@ -202,11 +203,4 @@
     </joint>
     <!-- end of joint list -->
-    <!-- ROS base_link to ABB base coordinate system transform -->
-    <link name="${prefix}base" />
-    <joint name="${prefix}base_link-base" type="fixed">
-      <origin xyz="0 0 0" rpy="0 0 0"/>
-      <parent link="${prefix}base_link"/>
-      <child link="${prefix}base"/>
-    </joint>
   </xacro:macro>
 </robot>

File: zoo/processed/ABB/IRB6640/xacro/irb6640_185_280_macro.xacro (robot description, xacro)
@@ -96,5 +96,7 @@
       </visual>
     </link>
-    <link name="${prefix}tool0"/>
+    <link name="${prefix}tool0">
+        <bow tags="effector"/>
+    </link>
     <!--Cylinder and piston -->
     <link name="${prefix}link_cylinder">
@@ -123,5 +125,4 @@
         <material name="yellow"/>
       </visual>
-      <bow name="arm" functions="goto point"/>
     </link>
     <!-- end of link list -->
