Commit message: Universal Robots bow tags

File: zoo/processed/Universal Robot/UR10/xacro/inc/ur_macro.xacro (robot description, xacro)
@@ -309,5 +309,7 @@
     </joint>
     <!-- ROS-Industrial 'tool0' frame: all-zeros tool frame -->
-    <link name="${prefix}tool0"/>
+    <link name="${prefix}tool0">
+        <bow tags="effector"/>
+    </link>
     <joint name="${prefix}flange-tool0" type="fixed">
       <!-- default toolframe: X+ left, Y+ up, Z+ front -->
