Commit message: BOW tagging extravaganza

File: zoo/processed/Fanuc/CR35IA/xacro/cr35ia_macro.xacro (robot description, xacro)
@@ -169,5 +169,7 @@
     </joint>
     <!-- ROS-Industrial 'tool0' frame: all-zeros tool frame -->
-    <link name="${prefix}tool0" />
+    <link name="${prefix}tool0">
+        <bow tags="effector"/>
+    </link>
     <joint name="${prefix}link_6-tool0" type="fixed">
       <origin xyz="0 0 0" rpy="${pi} ${-pi/2.0} 0" />

File: zoo/processed/Fanuc/CR7IA/xacro/cr7ia_macro.xacro (robot description, xacro)
@@ -167,5 +167,7 @@
     </joint>
     <!-- ROS-Industrial 'tool0' frame: all-zeros tool frame -->
-    <link name="${prefix}tool0" />
+    <link name="${prefix}tool0">
+        <bow tags="effector"/>
+    </link>
     <joint name="${prefix}link_6-tool0" type="fixed">
       <origin xyz="0 0 0" rpy="${pi} ${-pi/2.0} 0" />

File: zoo/processed/Fanuc/CR7IAL/xacro/cr7ial_macro.xacro (robot description, xacro)
@@ -167,5 +167,7 @@
     </joint>
     <!-- ROS-Industrial 'tool0' frame: all-zeros tool frame -->
-    <link name="${prefix}tool0" />
+    <link name="${prefix}tool0">
+        <bow tags="effector"/>
+    </link>
     <joint name="${prefix}link_6-tool0" type="fixed">
       <origin xyz="0 0 0" rpy="${pi} ${-pi/2.0} 0" />

File: zoo/processed/Fanuc/LRMate200i/xacro/lrmate200i_macro.xacro (robot description, xacro)
@@ -167,5 +167,7 @@
     </joint>
     <!-- ROS-Industrial 'tool0' frame: all-zeros tool frame -->
-    <link name="${prefix}tool0" />
+    <link name="${prefix}tool0">
+        <bow tags="effector"/>
+    </link>
     <joint name="${prefix}link_6-tool0" type="fixed">
       <origin xyz="0 0 0" rpy="${pi} ${-pi/2.0} 0" />

File: zoo/processed/Fanuc/LRMate200ib/xacro/lrmate200ib_macro.xacro (robot description, xacro)
@@ -167,5 +167,7 @@
     </joint>
     <!-- ROS-Industrial 'tool0' frame: all-zeros tool frame -->
-    <link name="${prefix}tool0" />
+    <link name="${prefix}tool0">
+        <bow tags="effector"/>
+    </link>
     <joint name="${prefix}link_6-tool0" type="fixed">
       <origin xyz="0 0 0" rpy="${pi} ${-pi/2.0} 0" />

File: zoo/processed/Fanuc/LRMate200ib3l/xacro/lrmate200ib3l_macro.xacro (robot description, xacro)
@@ -167,5 +167,7 @@
     </joint>
     <!-- ROS-Industrial 'tool0' frame: all-zeros tool frame -->
-    <link name="${prefix}tool0" />
+    <link name="${prefix}tool0">
+        <bow tags="effector"/>
+    </link>
     <joint name="${prefix}link_6-tool0" type="fixed">
       <origin xyz="0 0 0" rpy="${pi} ${-pi/2.0} 0" />

File: zoo/processed/Fanuc/LRMate200ic/xacro/lrmate200ic_macro.xacro (robot description, xacro)
@@ -167,5 +167,7 @@
     </joint>
     <!-- ROS-Industrial 'tool0' frame: all-zeros tool frame -->
-    <link name="${prefix}tool0" />
+    <link name="${prefix}tool0">
+        <bow tags="effector"/>
+    </link>
     <joint name="${prefix}link_6-tool0" type="fixed">
       <origin xyz="0 0 0" rpy="${pi} ${-pi/2.0} 0" />

File: zoo/processed/Fanuc/LRMate200ic5f/xacro/lrmate200ic5f_macro.xacro (robot description, xacro)
@@ -145,5 +145,7 @@
     </joint>
     <!-- ROS-Industrial 'tool0' frame: all-zeros tool frame -->
-    <link name="${prefix}tool0" />
+    <link name="${prefix}tool0">
+        <bow tags="effector"/>
+    </link>
     <joint name="${prefix}link_5-tool0" type="fixed">
       <origin xyz="0 0 0" rpy="${pi} ${-pi/2.0} 0" />

File: zoo/processed/Fanuc/LRMate200ic5h/xacro/lrmate200ic5h_macro.xacro (robot description, xacro)
@@ -145,5 +145,7 @@
     </joint>
     <!-- ROS-Industrial 'tool0' frame: all-zeros tool frame -->
-    <link name="${prefix}tool0" />
+    <link name="${prefix}tool0">
+        <bow tags="effector"/>
+    </link>
     <joint name="${prefix}link_5-tool0" type="fixed">
       <origin xyz="0 0 0" rpy="${pi} ${-pi/2.0} 0" />

File: zoo/processed/Fanuc/LRMate200ic5hs/xacro/lrmate200ic5hs_macro.xacro (robot description, xacro)
@@ -145,5 +145,7 @@
     </joint>
     <!-- ROS-Industrial 'tool0' frame: all-zeros tool frame -->
-    <link name="${prefix}tool0" />
+    <link name="${prefix}tool0">
+        <bow tags="effector"/>
+    </link>
     <joint name="${prefix}link_5-tool0" type="fixed">
       <origin xyz="0 0 0" rpy="${pi} ${-pi/2.0} 0" />

File: zoo/processed/Fanuc/LRMate200ic5l/xacro/lrmate200ic5l_macro.xacro (robot description, xacro)
@@ -167,5 +167,7 @@
     </joint>
     <!-- ROS-Industrial 'tool0' frame: all-zeros tool frame -->
-    <link name="${prefix}tool0" />
+    <link name="${prefix}tool0">
+        <bow tags="effector"/>
+    </link>
     <joint name="${prefix}link_6-tool0" type="fixed">
       <origin xyz="0 0 0" rpy="${pi} ${-pi/2.0} 0" />

File: zoo/processed/Fanuc/LRMate200id/xacro/lrmate200id_macro.xacro (robot description, xacro)
@@ -167,5 +167,7 @@
     </joint>
     <!-- ROS-Industrial 'tool0' frame: all-zeros tool frame -->
-    <link name="${prefix}tool0" />
+    <link name="${prefix}tool0">
+        <bow tags="effector"/>
+    </link>
     <joint name="${prefix}flange-tool0" type="fixed">
       <origin xyz="0 0 0" rpy="${pi} ${-pi/2.0} 0" />

File: zoo/processed/Fanuc/LRMate200id4s/xacro/lrmate200id4s_macro.xacro (robot description, xacro)
@@ -167,5 +167,7 @@
     </joint>
     <!-- ROS-Industrial 'tool0' frame: all-zeros tool frame -->
-    <link name="${prefix}tool0" />
+    <link name="${prefix}tool0">
+        <bow tags="effector"/>
+    </link>
     <joint name="${prefix}flange-tool0" type="fixed">
       <origin xyz="0 0 0" rpy="${pi} ${-pi/2.0} 0" />

File: zoo/processed/Fanuc/LRMate200id4sc/xacro/lrmate200id4sc_macro.xacro (robot description, xacro)
@@ -167,5 +167,7 @@
     </joint>
     <!-- ROS-Industrial 'tool0' frame: all-zeros tool frame -->
-    <link name="${prefix}tool0" />
+    <link name="${prefix}tool0">
+        <bow tags="effector"/>
+    </link>
     <joint name="${prefix}flange-tool0" type="fixed">
       <origin xyz="0 0 0" rpy="${pi} ${-pi/2.0} 0" />

File: zoo/processed/Fanuc/LRMate200id4sh/xacro/lrmate200id4sh_macro.xacro (robot description, xacro)
@@ -161,5 +161,7 @@
     </joint>
     <!-- ROS-Industrial 'tool0' frame: all-zeros tool frame -->
-    <link name="${prefix}tool0" />
+    <link name="${prefix}tool0">
+        <bow tags="effector"/>
+    </link>
     <joint name="${prefix}flange-tool0" type="fixed">
       <origin xyz="0 0 0" rpy="${pi} ${-pi/2.0} 0" />

File: zoo/processed/Fanuc/LRMate200id7h/xacro/lrmate200id7h_macro.xacro (robot description, xacro)
@@ -161,5 +161,7 @@
     </joint>
     <!-- ROS-Industrial 'tool0' frame: all-zeros tool frame -->
-    <link name="${prefix}tool0" />
+    <link name="${prefix}tool0">
+        <bow tags="effector"/>
+    </link>
     <joint name="${prefix}flange-tool0" type="fixed">
       <origin xyz="0 0 0" rpy="${pi} ${-pi/2.0} 0" />

File: zoo/processed/Fanuc/LRMate200id7l/xacro/lrmate200id7l_macro.xacro (robot description, xacro)
@@ -167,5 +167,7 @@
     </joint>
     <!-- ROS-Industrial 'tool0' frame: all-zeros tool frame -->
-    <link name="${prefix}tool0" />
+    <link name="${prefix}tool0">
+        <bow tags="effector"/>
+    </link>
     <joint name="${prefix}flange-tool0" type="fixed">
       <origin xyz="0 0 0" rpy="${pi} ${-pi/2.0} 0" />

File: zoo/processed/Fanuc/LRMate200id7lc/xacro/lrmate200id7lc_macro.xacro (robot description, xacro)
@@ -167,5 +167,7 @@
     </joint>
     <!-- ROS-Industrial 'tool0' frame: all-zeros tool frame -->
-    <link name="${prefix}tool0" />
+    <link name="${prefix}tool0">
+        <bow tags="effector"/>
+    </link>
     <joint name="${prefix}flange-tool0" type="fixed">
       <origin xyz="0 0 0" rpy="${pi} ${-pi/2.0} 0" />

File: zoo/processed/Fanuc/M10ia/xacro/m10ia_macro.xacro (robot description, xacro)
@@ -167,5 +167,7 @@
     </joint>
     <!-- ROS-Industrial 'tool0' frame: all-zeros tool frame -->
-    <link name="${prefix}tool0" />
+    <link name="${prefix}tool0">
+        <bow tags="effector"/>
+    </link>
     <joint name="${prefix}link_6-tool0" type="fixed">
       <origin xyz="0 0 0" rpy="${pi} ${-pi/2.0} 0" />

File: zoo/processed/Fanuc/M10ia7l/xacro/m10ia7l_macro.xacro (robot description, xacro)
@@ -167,5 +167,7 @@
     </joint>
     <!-- ROS-Industrial 'tool0' frame: all-zeros tool frame -->
-    <link name="${prefix}tool0" />
+    <link name="${prefix}tool0">
+        <bow tags="effector"/>
+    </link>
     <joint name="${prefix}link_6-tool0" type="fixed">
       <origin xyz="0 0 0" rpy="${pi} ${-pi/2.0} 0" />
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