Commit message: bluerov updates

File: zoo/processed/Blue Robotics/BlueROV2_Reach/bluerov2_reach.urdf (robot description, URDF)
Before this commit: robot reach5mini, 10 links, 9 joints
Links:
- link rov_base_link: geometry collision mesh filename=meshes/reach5mini/visual/BlueRov2.dae; visual mesh filename=meshes/reach5mini/visual/BlueRov2.dae

Commit message: Bluerov changes

File: zoo/processed/Blue Robotics/BlueROV2_Reach/bluerov2_reach.urdf (robot description, URDF)
Before this commit: robot reach5mini, 10 links, 9 joints
Links:
- link rov_base_link: geometry collision mesh filename=meshes/reach5mini/visual/bluerov2_noprop.dae; visual mesh filename=meshes/reach5mini/visual/bluerov2_noprop.dae
