Commit message: youbot urdf fix

File: zoo/processed/KUKA/youBot/xacro/youbot_arm/arm.urdf.xacro (robot description, xacro)
@@ -61,7 +61,7 @@
 			</inertial>
 			<visual>
-				<origin xyz="0 0 0" rpy="0 0 0" />
-				<geometry>
-					<mesh filename="package://youbot_description/meshes/youbot_arm/arm1.dae" />
+				<origin xyz="0 0 -0.045" rpy="0 0 0" />
+				<geometry>
+					<mesh filename="package://youbot_description/meshes/youbot_arm/arm1.dae" scale="0.0254 0.0254 0.0254"/>
 				</geometry>
 				<!--<material name="Orange" />-->
@@ -69,7 +69,7 @@
 			<collision>
 				<!--<origin xyz="0 0 -0.003" rpy="0 0 0" />-->
-				<origin xyz="0 0 0" rpy="0 0 0" />
-				<geometry>
-					<mesh filename="package://youbot_description/meshes/youbot_arm/arm1_convex.dae" />
+				<origin xyz="0 0 -0.045" rpy="0 0 0" />
+				<geometry>
+					<mesh filename="package://youbot_description/meshes/youbot_arm/arm1_convex.dae" scale="0.0254 0.0254 0.0254"/>
 					<!--<cylinder length="0.102" radius="0.080"/>-->
 				</geometry>
