Commit message: Fixed xacro for youbot2

File: zoo/processed/KUKA/youBot/xacro/youbot.xacro (robot description, xacro)
@@ -1,8 +1,4 @@
 <?xml version="1.0"?>
-<robot xmlns:sensor="http://playerstage.sourceforge.net/gazebo/xmlschema/#sensor"
-       xmlns:controller="http://playerstage.sourceforge.net/gazebo/xmlschema/#controller"
-       xmlns:interface="http://playerstage.sourceforge.net/gazebo/xmlschema/#interface"
-       xmlns:xacro="http://playerstage.sourceforge.net/gazebo/xmlschema/#interface"
-       name="youbot" >
+<robot name="youbot" xmlns:xacro="http://www.ros.org/wiki/xacro">
   <!-- The following included files set up definitions of parts of the robot body -->
   <!-- misc common stuff? -->

File: zoo/processed/KUKA/youbot2/xacro/youbot_arm/limits.urdf.xacro (robot description, xacro)
@@ -2,31 +2,31 @@
 <robot name="youbot" xmlns:xacro="http://ros.org/wiki/xacro">
 	<!-- common properties -->
-	<property name="M_PI" value="3.1415926535897931" />
+	<xacro:property name="M_PI" value="3.1415926535897931" />
 	<!--<property name="threshold" value="0.01" />-->
-	<property name="threshold" value="0.05" />
+	<xacro:property name="threshold" value="0.05" />
 	<!-- arm limits positions (deg)-->
-	<property name="joint_1_limit" value="${M_PI * (169 + 169) / 180}" />
-	<property name="joint_2_limit" value="${M_PI * (90 + 65) / 180}" />
-	<property name="joint_3_limit" value="${M_PI * (146 + 151) / 180}" />
-	<property name="joint_4_limit" value="${M_PI * (102.5 + 102.5) / 180}" />
-	<property name="joint_5_limit" value="${M_PI * (167.5 + 167.5) / 180}" />
-	<property name="joint_1_limit_soft" value="${M_PI * (169 + 169) / 180 - threshold}" />
-	<property name="joint_2_limit_soft" value="${M_PI * (90 + 65) / 180 - threshold}" />
-	<property name="joint_3_limit_soft" value="${M_PI * (146 + 151) / 180 - threshold}" />
-	<property name="joint_4_limit_soft" value="${M_PI * (102.5 + 102.5) / 180 - threshold}" />
-	<property name="joint_5_limit_soft" value="${M_PI * (167.5 + 167.5) / 180 - threshold}" />
+	<xacro:property name="joint_1_limit" value="${M_PI * (169 + 169) / 180}" />
+	<xacro:property name="joint_2_limit" value="${M_PI * (90 + 65) / 180}" />
+	<xacro:property name="joint_3_limit" value="${M_PI * (146 + 151) / 180}" />
+	<xacro:property name="joint_4_limit" value="${M_PI * (102.5 + 102.5) / 180}" />
+	<xacro:property name="joint_5_limit" value="${M_PI * (167.5 + 167.5) / 180}" />
+	<xacro:property name="joint_1_limit_soft" value="${M_PI * (169 + 169) / 180 - threshold}" />
+	<xacro:property name="joint_2_limit_soft" value="${M_PI * (90 + 65) / 180 - threshold}" />
+	<xacro:property name="joint_3_limit_soft" value="${M_PI * (146 + 151) / 180 - threshold}" />
+	<xacro:property name="joint_4_limit_soft" value="${M_PI * (102.5 + 102.5) / 180 - threshold}" />
+	<xacro:property name="joint_5_limit_soft" value="${M_PI * (167.5 + 167.5) / 180 - threshold}" />
 	<!-- dynamic properties : mass (kg) Alu data sheet -->
-	<property name="link_0_mass" value="0.845" />
-	<property name="link_1_mass" value="2.412" />
-	<property name="link_2_mass" value="1.155" />
-	<property name="link_3_mass" value="0.934" />
-	<property name="link_4_mass" value="0.877" />
-	<property name="link_5_mass" value="0.251" />
+	<xacro:property name="link_0_mass" value="0.845" />
+	<xacro:property name="link_1_mass" value="2.412" />
+	<xacro:property name="link_2_mass" value="1.155" />
+	<xacro:property name="link_3_mass" value="0.934" />
+	<xacro:property name="link_4_mass" value="0.877" />
+	<xacro:property name="link_5_mass" value="0.251" />
 	<!--<property name="link_0_mass" value="0.845" />
-	<property name="link_1_mass" value="0.1" />
-	<property name="link_2_mass" value="0.1" />
-	<property name="link_3_mass" value="0.1" />
-	<property name="link_4_mass" value="0.1" />
-	<property name="link_5_mass" value="0.1" />-->
+	<xacro:property name="link_1_mass" value="0.1" />
+	<xacro:property name="link_2_mass" value="0.1" />
+	<xacro:property name="link_3_mass" value="0.1" />
+	<xacro:property name="link_4_mass" value="0.1" />
+	<xacro:property name="link_5_mass" value="0.1" />-->
 	<!-- TODO: add inertia tensor-->
 	<xacro:macro name="default_origin">

File: zoo/processed/KUKA/youbot2/xacro/youbot_base/base.transmission.xacro (robot description, xacro)
@@ -1,7 +1,7 @@
 <?xml version="1.0"?>
 <robot name="youbot" xmlns:xacro="http://www.ros.org/wiki/xacro">
-  <property name="wheel_mechanical_reduction" value="${624/35 * 80/18}"/>
-  <property name="caster_mechanical_reduction" value="${624/35 * 80/18}"/>
-  <property name="" value="0.360"/>
+  <xacro:property name="wheel_mechanical_reduction" value="${624/35 * 80/18}"/>
+  <xacro:property name="caster_mechanical_reduction" value="${624/35 * 80/18}"/>
+  <xacro:property name="random" value="0.360"/>
   <xacro:macro name="youbot_base_transmission">
     <!-- front left wheel -->

File: zoo/processed/KUKA/youbot2/xacro/youbot_base/base.urdf.xacro (robot description, xacro)
@@ -6,28 +6,28 @@
   <xacro:include filename="$(find youbot_description)/urdf/youbot_base/base.transmission.xacro" />
   <!-- simplified box collision geometry for base -->
-  <property name="base_size_x" value="0.570" />
-  <property name="base_size_y" value="0.360" />
-  <property name="base_size_z" value="0.100" />
-  <property name="base_mass" value="22.0" />
-  <property name="caster_offset_x" value="0.228"  />
-  <property name="caster_offset_y" value="0.158"  />
-  <property name="caster_offset_z" value="-0.034" />
-  <property name="caster_mass" value="0.1" />
-  <property name="wheel_offset_x" value="0.0"  />
-  <property name="wheel_offset_y" value="0.0"  />
-  <property name="wheel_offset_z" value="0.0" />
-  <property name="wheel_mass" value="0.4" />
-  <property name="wheel_radius" value="0.05" />
-  <property name="wheel_length" value="0.005" />
-  <property name="caster_joint_damping" value="1.0" />
-  <property name="caster_joint_friction" value="1.0" />
-  <property name="caster_joint_effort" value="30" />
-  <property name="caster_joint_velocity" value="10" />
-  <property name="caster_joint_safety_k_velocity" value="10.0" />
-  <property name="wheel_joint_damping" value="1.0" />
-  <property name="wheel_joint_friction" value="1.0" />
-  <property name="wheel_joint_effort" value="30" />
-  <property name="wheel_joint_velocity" value="10" />
-  <property name="wheel_joint_safety_k_velocity" value="10.0" />
+  <xacro:property name="base_size_x" value="0.570" />
+  <xacro:property name="base_size_y" value="0.360" />
+  <xacro:property name="base_size_z" value="0.100" />
+  <xacro:property name="base_mass" value="22.0" />
+  <xacro:property name="caster_offset_x" value="0.228"  />
+  <xacro:property name="caster_offset_y" value="0.158"  />
+  <xacro:property name="caster_offset_z" value="-0.034" />
+  <xacro:property name="caster_mass" value="0.1" />
+  <xacro:property name="wheel_offset_x" value="0.0"  />
+  <xacro:property name="wheel_offset_y" value="0.0"  />
+  <xacro:property name="wheel_offset_z" value="0.0" />
+  <xacro:property name="wheel_mass" value="0.4" />
+  <xacro:property name="wheel_radius" value="0.05" />
+  <xacro:property name="wheel_length" value="0.005" />
+  <xacro:property name="caster_joint_damping" value="1.0" />
+  <xacro:property name="caster_joint_friction" value="1.0" />
+  <xacro:property name="caster_joint_effort" value="30" />
+  <xacro:property name="caster_joint_velocity" value="10" />
+  <xacro:property name="caster_joint_safety_k_velocity" value="10.0" />
+  <xacro:property name="wheel_joint_damping" value="1.0" />
+  <xacro:property name="wheel_joint_friction" value="1.0" />
+  <xacro:property name="wheel_joint_effort" value="30" />
+  <xacro:property name="wheel_joint_velocity" value="10" />
+  <xacro:property name="wheel_joint_safety_k_velocity" value="10.0" />
   <xacro:macro name="youbot_base" params="name">
     <link name="${name}_footprint">

File: zoo/processed/KUKA/youbot2/xacro/youbot_gripper/limits.urdf.xacro (robot description, xacro)
@@ -1,9 +1,9 @@
 <?xml version="1.0"?>
-<robot>
+<robot name="youbot" xmlns:xacro="http://ros.org/wiki/xacro">
 	<!-- common properties -->
-	<property name="M_PI" value="3.1415926535897931" />
-        <property name="gripper_threshold" value="0.001" />
+	<xacro:property name="M_PI" value="3.1415926535897931" />
+        <xacro:property name="gripper_threshold" value="0.001" />
 	<!-- fingers limits, values are in meters -->
-	<property name="finger_joint" value="${0.023 / 2.0}" />
-	<property name="finger_joint_soft" value="${(0.023 - gripper_threshold) / 2.0}" />
+	<xacro:property name="finger_joint" value="${0.023 / 2.0}" />
+	<xacro:property name="finger_joint_soft" value="${(0.023 - gripper_threshold) / 2.0}" />
 </robot>
