Commit message: Gripper xacro update and base mesh update for youbot

File: zoo/processed/KUKA/youbot2/xacro/youbot_gripper/gripper.urdf.xacro (robot description, xacro)
@@ -14,10 +14,10 @@
 		<link name="${name}_palm_link">
 			<inertial>
-				<origin xyz="0 0 0" rpy="${M_PI} ${-M_PI / 2}  0"/>
+				<origin xyz="0 0 0" rpy="${M_PI} ${M_PI}  0"/>
 				<mass value="0.1"/>
 				<inertia ixx="0.01" ixy="0" ixz="0" iyy="0.01" iyz="0" izz="0.01" />
 			</inertial>
 			<visual>
-				<origin xyz="0 0 0" rpy="${M_PI} ${-M_PI / 2} 0" />
+				<origin xyz="0.0025 0 0" rpy="${M_PI} ${M_PI} 0" />
 				<geometry>
 					<mesh filename="package://youbot_description/meshes/youbot_gripper/palm.dae" />
@@ -25,5 +25,5 @@
 			</visual>
 			<collision>
-				<origin xyz="0 0 0" rpy="${M_PI} ${-M_PI / 2} 0" />
+				<origin xyz="0.0025 0 0" rpy="${M_PI} ${M_PI} 0" />
 				<geometry>
 					<!--<box size="0.050 0.094 0.054"/>-->
@@ -51,5 +51,5 @@
 	-->
 	<joint name="${name}_finger_joint_l" type="prismatic">
-		<origin xyz="0.046 0.010 0.003 " rpy="0 ${-M_PI / 2} ${M_PI}" />
+		<origin xyz="0 0 0.003 " rpy="0 ${-M_PI / 2} ${M_PI}" />
 		<parent link="${name}_palm_link"/>
 		<child link="${name}_finger_link_l"/>
@@ -61,10 +61,10 @@
 	<link name="${name}_finger_link_l">
 		<inertial>
-			<origin xyz="0 -0.001 0" rpy="0 0 0" />
+			<origin xyz="0 ${M_PI / 2} 0" rpy="0 0 0" />
 			<mass value="0.01"/>
 			<inertia ixx="0.01" ixy="0" ixz="0" iyy="0.01" iyz="0" izz="0.01" />
 		</inertial>
 		<visual>
-			<origin xyz="0 0 0" rpy="0 0 0" />
+			<origin xyz="0 ${M_PI / 2} 0" rpy="0 0 0" />
 			<geometry>
 				<mesh filename="package://youbot_description/meshes/youbot_gripper/finger.dae" />
@@ -72,5 +72,5 @@
 		</visual>
 		<collision>
-			<origin xyz="0 0 0" rpy="0 0 0" />
+			<origin xyz="0 ${M_PI / 2} 0" rpy="0 0 0" />
 			<geometry>
 				<!--<box size="0.014 0.020 0.046"/>-->
@@ -80,5 +80,5 @@
 	</link>
 	<joint name="${name}_finger_joint_r" type="prismatic">
-		<origin xyz="0.046 -0.010 0.003" rpy="0 ${M_PI / 2} 0" />
+		<origin xyz="0 0 0.03" rpy="0 ${M_PI / 2} 0" />
 		<parent link="${name}_palm_link"/>
 		<child link="${name}_finger_link_r"/>
@@ -90,10 +90,10 @@
 	<link name="${name}_finger_link_r">
 		<inertial>
-			<origin xyz="0.000 -0.001 0" rpy="0 0 0" />
+			<origin xyz="0.000 ${-M_PI / 2} 0" rpy="0 0 0" />
 			<mass value="0.01"/>
 			<inertia ixx="0.01" ixy="0" ixz="0" iyy="0.01" iyz="0" izz="0.01" />
 		</inertial>
 		<visual>
-			<origin xyz="0 0 0" rpy="0 0 0" />
+			<origin xyz="0 ${-M_PI / 2} 0" rpy="0 0 0" />
 			<geometry>
 				<mesh filename="package://youbot_description/meshes/youbot_gripper/finger.dae" />
@@ -101,5 +101,5 @@
 		</visual>
 		<collision>
-			<origin xyz="0.000 0 0" rpy="0 0 0" />
+			<origin xyz="0.000 ${-M_PI / 2} 0" rpy="0 0 0" />
 			<geometry>
 				<!--<box size="0.014 0.020 0.046"/>-->

Commit message: gripper xacro update

File: zoo/processed/KUKA/youbot2/xacro/youbot_gripper/gripper.urdf.xacro (robot description, xacro)
@@ -51,5 +51,5 @@
 	-->
 	<joint name="${name}_finger_joint_l" type="prismatic">
-		<origin xyz="0 0 0.003 " rpy="0 ${-M_PI / 2} ${M_PI}" />
+		<origin xyz="0 0 0.03 " rpy="0 ${-M_PI / 2} ${M_PI}" />
 		<parent link="${name}_palm_link"/>
 		<child link="${name}_finger_link_l"/>
@@ -61,10 +61,10 @@
 	<link name="${name}_finger_link_l">
 		<inertial>
-			<origin xyz="0 ${M_PI / 2} 0" rpy="0 0 0" />
+			<origin xyz="0 0 0" rpy="0 ${M_PI / 2} 0" />
 			<mass value="0.01"/>
 			<inertia ixx="0.01" ixy="0" ixz="0" iyy="0.01" iyz="0" izz="0.01" />
 		</inertial>
 		<visual>
-			<origin xyz="0 ${M_PI / 2} 0" rpy="0 0 0" />
+			<origin xyz="0 0 0" rpy="0 ${M_PI / 2} 0" />
 			<geometry>
 				<mesh filename="package://youbot_description/meshes/youbot_gripper/finger.dae" />
@@ -72,5 +72,5 @@
 		</visual>
 		<collision>
-			<origin xyz="0 ${M_PI / 2} 0" rpy="0 0 0" />
+			<origin xyz="0 0 0" rpy="0 ${M_PI / 2} 0" />
 			<geometry>
 				<!--<box size="0.014 0.020 0.046"/>-->
@@ -90,10 +90,10 @@
 	<link name="${name}_finger_link_r">
 		<inertial>
-			<origin xyz="0.000 ${-M_PI / 2} 0" rpy="0 0 0" />
+			<origin xyz="0 0 0" rpy="0 ${-M_PI / 2}  0" />
 			<mass value="0.01"/>
 			<inertia ixx="0.01" ixy="0" ixz="0" iyy="0.01" iyz="0" izz="0.01" />
 		</inertial>
 		<visual>
-			<origin xyz="0 ${-M_PI / 2} 0" rpy="0 0 0" />
+			<origin xyz="0 0 0" rpy="0 ${-M_PI / 2}  0" />
 			<geometry>
 				<mesh filename="package://youbot_description/meshes/youbot_gripper/finger.dae" />
@@ -101,5 +101,5 @@
 		</visual>
 		<collision>
-			<origin xyz="0.000 ${-M_PI / 2} 0" rpy="0 0 0" />
+			<origin xyz="0 0 0" rpy="0 ${-M_PI / 2}  0" />
 			<geometry>
 				<!--<box size="0.014 0.020 0.046"/>-->

Commit message: yet another youbot update

File: zoo/processed/KUKA/youbot2/xacro/youbot_gripper/gripper.urdf.xacro (robot description, xacro)
@@ -51,5 +51,5 @@
 	-->
 	<joint name="${name}_finger_joint_l" type="prismatic">
-		<origin xyz="0 0 0.03 " rpy="0 ${-M_PI / 2} ${M_PI}" />
+		<origin xyz="0 0 0" rpy="0 0 ${M_PI}" />
 		<parent link="${name}_palm_link"/>
 		<child link="${name}_finger_link_l"/>
@@ -61,10 +61,10 @@
 	<link name="${name}_finger_link_l">
 		<inertial>
-			<origin xyz="0 0 0" rpy="0 ${M_PI / 2} 0" />
+			<origin xyz="0 -0.01 0" rpy="0 0 0" />
 			<mass value="0.01"/>
 			<inertia ixx="0.01" ixy="0" ixz="0" iyy="0.01" iyz="0" izz="0.01" />
 		</inertial>
 		<visual>
-			<origin xyz="0 0 0" rpy="0 ${M_PI / 2} 0" />
+			<origin xyz="0 -0.01 0" rpy="0 0} 0" />
 			<geometry>
 				<mesh filename="package://youbot_description/meshes/youbot_gripper/finger.dae" />
@@ -72,5 +72,5 @@
 		</visual>
 		<collision>
-			<origin xyz="0 0 0" rpy="0 ${M_PI / 2} 0" />
+			<origin xyz="0 -0.01 0" rpy="0 0 0" />
 			<geometry>
 				<!--<box size="0.014 0.020 0.046"/>-->
@@ -90,5 +90,5 @@
 	<link name="${name}_finger_link_r">
 		<inertial>
-			<origin xyz="0 0 0" rpy="0 ${-M_PI / 2}  0" />
+			<origin xyz="0 -0.01 0" rpy="0 ${-M_PI / 2}  0" />
 			<mass value="0.01"/>
 			<inertia ixx="0.01" ixy="0" ixz="0" iyy="0.01" iyz="0" izz="0.01" />
@@ -101,5 +101,5 @@
 		</visual>
 		<collision>
-			<origin xyz="0 0 0" rpy="0 ${-M_PI / 2}  0" />
+			<origin xyz="0 -0.01 0" rpy="0 ${-M_PI / 2}  0" />
 			<geometry>
 				<!--<box size="0.014 0.020 0.046"/>-->

Commit message: youbot update

File: zoo/processed/KUKA/youbot2/xacro/youbot_gripper/gripper.urdf.xacro (robot description, xacro)
@@ -61,10 +61,10 @@
 	<link name="${name}_finger_link_l">
 		<inertial>
-			<origin xyz="0 -0.01 0" rpy="0 0 0" />
+			<origin xyz="0 -0.01 0.03" rpy="0 0 0" />
 			<mass value="0.01"/>
 			<inertia ixx="0.01" ixy="0" ixz="0" iyy="0.01" iyz="0" izz="0.01" />
 		</inertial>
 		<visual>
-			<origin xyz="0 -0.01 0" rpy="0 0} 0" />
+			<origin xyz="0 -0.01 0.03" rpy="0 0} 0" />
 			<geometry>
 				<mesh filename="package://youbot_description/meshes/youbot_gripper/finger.dae" />
@@ -72,5 +72,5 @@
 		</visual>
 		<collision>
-			<origin xyz="0 -0.01 0" rpy="0 0 0" />
+			<origin xyz="0 -0.01 0.03" rpy="0 0 0" />
 			<geometry>
 				<!--<box size="0.014 0.020 0.046"/>-->
@@ -95,5 +95,5 @@
 		</inertial>
 		<visual>
-			<origin xyz="0 0 0" rpy="0 ${-M_PI / 2}  0" />
+			<origin xyz="0 -0.01 0" rpy="0 ${-M_PI / 2}  0" />
 			<geometry>
 				<mesh filename="package://youbot_description/meshes/youbot_gripper/finger.dae" />
