Commit message: Talos update

File: zoo/processed/PAL Robotics/Ari/xacro/torso/torso_sensors.urdf.xacro (robot description, xacro)
@@ -65,5 +65,5 @@
   <!-- Torso sensors -->
   <!-- Torso front camera -->
-  <xacro:sensor_d435 parent="${parent}" name="${name}_front_camera" topics_ns="${name}_front_camera" use_nominal_extrinsics="${use_nominal_extrinsics}">
+  <xacro:sensor_d435 parent="${parent}" name="${name}_front_camera" topics_ns="${name}_front_camera">
     <origin xyz="${torso_front_camera_position_x} ${torso_front_camera_position_y} ${torso_front_camera_position_z}"
             rpy="${torso_front_camera_orientation_r} ${torso_front_camera_orientation_p} ${torso_front_camera_orientation_y}"/>

File: zoo/processed/PAL Robotics/Talos/xacro/arm/arm.urdf.xacro (robot description, xacro)
@@ -25,10 +25,5 @@
   <xacro:property name="arm_eps"            value="0.02" />
   <xacro:macro name="talos_arm" params="name parent side reflect">
-    <xacro:unless value="$(arg test)">
-      <xacro:include filename="$(find talos_description_calibration)/urdf/calibration/arm_${side}.xacro" />
-    </xacro:unless>
-    <xacro:if value="$(arg test)">
-      <xacro:include filename="$(find talos_description)/test/calibration/arm_${side}.xacro" />
-    </xacro:if>
+  <xacro:include filename="$(find talos_description_calibration)/urdf/calibration/arm_${side}.xacro" />
     <!--************************-->
     <!--        SHOULDER        -->

File: zoo/processed/PAL Robotics/Talos/xacro/arm/wrist.urdf.xacro (robot description, xacro)
@@ -22,10 +22,5 @@
   <xacro:property name="wrist_eps"          value="0.02" />
   <xacro:macro name="talos_wrist" params="name parent side reflect">
-    <xacro:unless value="$(arg test)">
-      <xacro:include filename="$(find talos_description_calibration)/urdf/calibration/arm_${side}.xacro" />
-    </xacro:unless>
-    <xacro:if value="$(arg test)">
-      <xacro:include filename="$(find talos_description)/test/calibration/arm_${side}.xacro" />
-    </xacro:if>
+    <xacro:include filename="$(find talos_description_calibration)/urdf/calibration/arm_${side}.xacro" />
     <!--************************-->
     <!--        WRIST           -->

File: zoo/processed/PAL Robotics/Talos/xacro/deg_to_rad.xacro (robot description, xacro)
@@ -1,3 +1,3 @@
 <robot xmlns:xacro="http://ros.org/wiki/xacro">
-    <xacro:property name="deg_to_rad" value="0.01745329251994329577" />
+	<xacro:property name="deg_to_rad" value="0.01745329251994329577" />
 </robot>

File: zoo/processed/PAL Robotics/Talos/xacro/leg/leg.urdf.xacro (robot description, xacro)
@@ -10,10 +10,5 @@
   <xacro:property name="leg_damping"      value="0.0" />
   <xacro:macro name="talos_leg" params="prefix reflect flexibility:=false">
-    <xacro:unless value="$(arg test)">
-      <xacro:include filename="$(find talos_description_calibration)/urdf/calibration/leg_${prefix}.xacro" />
-    </xacro:unless>
-    <xacro:if value="$(arg test)">
-      <xacro:include filename="$(find talos_description)/test/calibration/leg_${prefix}.xacro" />
-    </xacro:if>
+  <xacro:include filename="$(find talos_description_calibration)/urdf/calibration/leg_${prefix}.xacro" />
     <xacro:if value="${flexibility}">
   <!-- Joint flex_hip_y (mesh link) : child link flex_hip_x -> parent link base_link -->

File: zoo/processed/PAL Robotics/Talos/xacro/talos_full_v1.urdf.xacro (robot description, xacro)
@@ -11,10 +11,5 @@
         xmlns:controller="http://playerstage.sourceforge.net/gazebo/xmlschema/#controller"
         xmlns:interface="http://playerstage.sourceforge.net/gazebo/xmlschema/#interface">
-  <xacro:arg name="enable_crane" default="0"/> <!-- right-arm, no-arm -->
-  <xacro:arg name="foot_collision" default="default"/> <!-- default, tallbox, thinbox -->
-  <xacro:arg name="disable_gazebo_camera" default="false"/> <!-- false, true -->
-  <xacro:arg name="head_type" default="default"/> <!-- default, lidar -->
-  <xacro:arg name="flexibility" default="false"/> <!-- false, true -->
-  <xacro:include filename="$(find talos_description)/urdf/arm/arm_specifics_v2.urdf.xacro" />
+  <xacro:include filename="$(find talos_description)/urdf/arm/arm_specifics_v1.urdf.xacro" />
   <xacro:include filename="$(find talos_description)/urdf/talos_full_common.urdf.xacro" />
 </robot>

File: zoo/processed/PAL Robotics/Talos/xacro/torso/torso.urdf.xacro (robot description, xacro)
@@ -12,10 +12,5 @@
   <xacro:include filename="$(find talos_description)/urdf/torso/torso.transmission.xacro" />
   <xacro:include filename="$(find talos_description)/urdf/sensors/imu.urdf.xacro" />
-  <xacro:unless value="$(arg test)">
-    <xacro:include filename="$(find talos_description_calibration)/urdf/calibration/calibration_constants.urdf.xacro" />
-  </xacro:unless>
-  <xacro:if value="$(arg test)">
-    <xacro:include filename="$(find talos_description)/test/calibration/calibration_constants.urdf.xacro" />
-  </xacro:if>
+  <xacro:include filename="$(find talos_description_calibration)/urdf/calibration/calibration_constants.urdf.xacro" />
  <!--Constant parameters-->
   <xacro:property name="torso_max_vel"  value="5.4" />
