Commit message: Tiago dual update

File: zoo/processed/PAL Robotics/Tiago_Dual/xacro/calibration/calibration_constants.urdf.xacro (robot description, xacro)
@@ -1,18 +1,13 @@
 <?xml version="1.0"?>
 <!--
-Copyright (c) 2022 PAL Robotics S.L. All rights reserved.
-Licensed under the Apache License, Version 2.0 (the "License");
-you may not use this file except in compliance with the License.
-You may obtain a copy of the License at
-    http://www.apache.org/licenses/LICENSE-2.0
-Unless required by applicable law or agreed to in writing, software
-distributed under the License is distributed on an "AS IS" BASIS,
-WITHOUT WARRANTIES OR CONDITIONS OF ANY KIND, either express or implied.
-See the License for the specific language governing permissions and
-limitations under the License.
- -->
+  Copyright (c) 2015, PAL Robotics, S.L.
+  All rights reserved.
+  This work is licensed under the Creative Commons Attribution-NonCommercial-NoDerivs 3.0 Unported License.
+  To view a copy of this license, visit http://creativecommons.org/licenses/by-nc-nd/3.0/ or send a letter to
+  Creative Commons, 444 Castro Street, Suite 900, Mountain View, California, 94041, USA.
+-->
 <robot xmlns:xacro="http://ros.org/wiki/xacro">
   <!--File includes-->
-  <xacro:include filename="$(find pal_urdf_utils)/urdf/deg_to_rad.urdf.xacro" />
+  <xacro:include filename="$(find tiago_dual_description_calibration)/urdf/deg_to_rad.xacro" />
   <!--Constant parameters-->
   <xacro:property name="camera_position_x" value="0.0908" />
@@ -22,11 +17,18 @@
   <xacro:property name="camera_orientation_p" value="0.0" />
   <xacro:property name="camera_orientation_y" value="0.0" />
-  <xacro:property name="arm_1_joint_offset" value="0.0" />
-  <xacro:property name="arm_2_joint_offset" value="0.0" />
-  <xacro:property name="arm_3_joint_offset" value="0.0" />
-  <xacro:property name="arm_4_joint_offset" value="0.0" />
-  <xacro:property name="arm_5_joint_offset" value="0.0" />
-  <xacro:property name="arm_6_joint_offset" value="0.0" />
-  <xacro:property name="arm_7_joint_offset" value="0.0" />
+  <xacro:property name="arm_left_1_joint_offset" value="0.0" />
+  <xacro:property name="arm_left_2_joint_offset" value="0.0" />
+  <xacro:property name="arm_left_3_joint_offset" value="0.0" />
+  <xacro:property name="arm_left_4_joint_offset" value="0.0" />
+  <xacro:property name="arm_left_5_joint_offset" value="0.0" />
+  <xacro:property name="arm_left_6_joint_offset" value="0.0" />
+  <xacro:property name="arm_left_7_joint_offset" value="0.0" />
+  <xacro:property name="arm_right_1_joint_offset" value="0.0" />
+  <xacro:property name="arm_right_2_joint_offset" value="0.0" />
+  <xacro:property name="arm_right_3_joint_offset" value="0.0" />
+  <xacro:property name="arm_right_4_joint_offset" value="0.0" />
+  <xacro:property name="arm_right_5_joint_offset" value="0.0" />
+  <xacro:property name="arm_right_6_joint_offset" value="0.0" />
+  <xacro:property name="arm_right_7_joint_offset" value="0.0" />
   <xacro:property name="head_1_joint_offset" value="0.0" />
   <xacro:property name="head_2_joint_offset" value="0.0" />

File: zoo/processed/PAL Robotics/Tiago_Dual/xacro/calibration/extrinsic_camera_calibration_constants.urdf.xacro (robot description, xacro)
@@ -1,18 +1,13 @@
 <?xml version="1.0"?>
 <!--
-Copyright (c) 2022 PAL Robotics S.L. All rights reserved.
-Licensed under the Apache License, Version 2.0 (the "License");
-you may not use this file except in compliance with the License.
-You may obtain a copy of the License at
-    http://www.apache.org/licenses/LICENSE-2.0
-Unless required by applicable law or agreed to in writing, software
-distributed under the License is distributed on an "AS IS" BASIS,
-WITHOUT WARRANTIES OR CONDITIONS OF ANY KIND, either express or implied.
-See the License for the specific language governing permissions and
-limitations under the License.
- -->
+  Copyright (c) 2015, PAL Robotics, S.L.
+  All rights reserved.
+  This work is licensed under the Creative Commons Attribution-NonCommercial-NoDerivs 3.0 Unported License.
+  To view a copy of this license, visit http://creativecommons.org/licenses/by-nc-nd/3.0/ or send a letter to
+  Creative Commons, 444 Castro Street, Suite 900, Mountain View, California, 94041, USA.
+-->
 <robot xmlns:xacro="http://ros.org/wiki/xacro">
   <!--File includes-->
-  <xacro:include filename="$(find pal_urdf_utils)/urdf/deg_to_rad.urdf.xacro" />
+  <xacro:include filename="$(find tiago_dual_description_calibration)/urdf/deg_to_rad.xacro" />
 <xacro:macro name="camera_baseline_constants" params="camera_model" >
   <xacro:if value="${camera_model == 'orbbec-astra'}">

File: zoo/processed/PAL Robotics/Tiago_Dual/xacro/tiago_dual.xacro (robot description, xacro)
@@ -121,6 +121,5 @@
 	      <xacro:ft_sensor name="wrist_left" parent="arm_left_tool_link" />
 	  </xacro:if>
-  <xacro:tiago_end_effector name="${end_effector_left_name}" parent="${end_effector_left_link}" type="${end_effector_left}"
-    has_end_effector="${has_end_effector_left}" reflect="-1" is_dual="true"/>
+  <xacro:tiago_end_effector name="${end_effector_left_name}" parent="${end_effector_left_link}" type="${end_effector_left}" reflect="-1" />
   </xacro:if>
   <!-- Right -->
@@ -132,5 +131,5 @@
 	      <xacro:ft_sensor name="wrist_right" parent="arm_right_tool_link" />
 	  </xacro:if>
-	  <xacro:tiago_end_effector name="${end_effector_right_name}" parent="${end_effector_right_link}" type="${end_effector_right}" has_end_effector="${has_end_effector_right}" reflect="1" is_dual="true"/>
+	  <xacro:tiago_end_effector name="${end_effector_right_name}" parent="${end_effector_right_link}" type="${end_effector_right}" reflect="1" />
   </xacro:if>
   <!-- RGBD Laser Link -->
