Commit message: Mesh dir optional for Artus hands

File: zoo/processed/Sarcomere Dynamics/Artus Dex Left/xacro/artus_dex_left_macro.xacro (robot description, xacro)
@@ -1,5 +1,5 @@
 <?xml version="1.0" ?>
 <robot xmlns:xacro="http://ros.org/wiki/xacro">
-	<xacro:macro name="artus_dex_left" params="base_link mesh_dir">
+	<xacro:macro name="artus_dex_left" params="base_link mesh_dir:=''">
 		<joint name="virtual" type="fixed">
 			<origin xyz="0 0 0" rpy="0 0 0"/>

File: zoo/processed/Sarcomere Dynamics/Artus Dex Right/xacro/artus_dex_right_macro.xacro (robot description, xacro)
@@ -1,5 +1,5 @@
 <?xml version="1.0" ?>
 <robot xmlns:xacro="http://ros.org/wiki/xacro">
-	<xacro:macro name="artus_dex_right" params="base_link mesh_dir">
+	<xacro:macro name="artus_dex_right" params="base_link mesh_dir:=''">
 		<joint name="virtual" type="fixed">
 			<origin xyz="0 0 0" rpy="0 0 0"/>
