Commit message: Added contact and loco tags to tiago

File: zoo/processed/PAL Robotics/Tiago/xacro/base/base.urdf.xacro (robot description, xacro)
@@ -12,5 +12,5 @@
   limitations under the License.
  -->
-<robot xmlns:xacro="http://ros.org/wiki/xacro">
+<robot locomotion="differential" xmlns:xacro="http://ros.org/wiki/xacro">
   <xacro:include filename="$(find pal_urdf_utils)/urdf/deg_to_rad.urdf.xacro"/>
   <xacro:include filename="$(find pmb2_description)/urdf/wheels/wheel.urdf.xacro"/>

File: zoo/processed/PAL Robotics/Tiago/xacro/wheels/wheel.urdf.xacro (robot description, xacro)
@@ -14,5 +14,5 @@
 <robot xmlns:xacro="http://ros.org/wiki/xacro">
   <xacro:include filename="$(find pmb2_description)/urdf/wheels/wheel.gazebo.xacro"/>
-  <xacro:macro name="wheel" params="side reflect radius width torque velocity separation parent">
+  <xacro:macro name="wheel" contact="wheel" params="side reflect radius width torque velocity separation parent">
     <link name="wheel_${side}_link">
       <inertial>
