Commit message: Added cameras to lite3

File: zoo/processed/DEEP Robotics/Lite3/lite3.urdf (robot description, URDF)
Before this commit: robot Lite3, 17 links, 16 joints
Links:
- added link FrontCamera_frame
- added link RearCamera_frame
Joints:
- added joint FrontCamera_fixed_joint: type fixed, parent TORSO, child FrontCamera_frame, origin xyz=0.28 0 0 rpy=0 0 0, axis 0 0 0
- added joint RearCamera_fixed_joint: type fixed, parent TORSO, child RearCamera_frame, origin xyz=-0.28 0 0 rpy=0 0 3.141, axis 0 0 0

Commit message: Addition of foot bumpers for Lite3

File: zoo/processed/DEEP Robotics/Lite3/lite3.urdf (robot description, URDF)
Before this commit: robot Lite3, 19 links, 18 joints
Links:
- link FL_FOOT: geometry collision mesh filename=meshes/foot_bumper.dae; visual mesh filename=meshes/foot_bumper.dae
- link FR_FOOT: geometry collision mesh filename=meshes/foot_bumper.dae; visual mesh filename=meshes/foot_bumper.dae
- link HL_FOOT: geometry collision mesh filename=meshes/foot_bumper.dae; visual mesh filename=meshes/foot_bumper.dae
- link HR_FOOT: geometry collision mesh filename=meshes/foot_bumper.dae; visual mesh filename=meshes/foot_bumper.dae
