Commit message: Sarcomere Theia update

File: zoo/processed/Sarcomere Dynamics/Theia/xacro/artus_dex_left_macro.xacro (robot description, xacro)
@@ -311,4 +311,5 @@
 				<inertia ixx="0" ixy="0"  ixz="0" iyy="0" iyz="0" izz="0" />
 			</inertial>
+			<bow tags="effector"/>
 		</link>
 		<joint name="Lindex_34" type="revolute">
@@ -431,4 +432,5 @@
 				<inertia ixx="0" ixy="0"  ixz="0" iyy="0" iyz="0" izz="0" />
 			</inertial>
+			<bow tags="effector"/>
 		</link>
 		<joint name="Lring_34" type="revolute">
@@ -551,4 +553,5 @@
 				<inertia ixx="0" ixy="0"  ixz="0" iyy="0" iyz="0" izz="0" />
 			</inertial>
+			<bow tags="effector"/>
 		</link>
 		<joint name="Lmiddle_34" type="revolute">
@@ -670,5 +673,6 @@
 				<mass value="0" />
 				<inertia ixx="0" ixy="0"  ixz="0" iyy="0" iyz="0" izz="0" />
-		</inertial>
+			</inertial>
+			<bow tags="effector"/>
 		</link>
 		<joint name="Lpinky_34" type="revolute">
@@ -791,4 +795,5 @@
 				<inertia ixx="0" ixy="0"  ixz="0" iyy="0" iyz="0" izz="0" />
 			</inertial>
+			<bow tags="effector"/>
 		</link>
 		<joint name="Lthumb_34" type="revolute">

File: zoo/processed/Sarcomere Dynamics/Theia/xacro/elephantbot_mycobot320_macro.xacro (robot description, xacro)
@@ -1,12 +1,12 @@
 <?xml version="1.0" ?>
 <robot xmlns:xacro="http://ros.org/wiki/xacro">
-	<xacro:macro name="elephantbot_mycobot_pro_320" params="base_link">
-        <joint name="head_base_joint" type="fixed">
+	<xacro:macro name="elephantbot_mycobot_pro_320" params="base_link end_link">
+        <joint name="cobot_base_joint" type="fixed">
             <parent link="${base_link}"/>
-            <child link="head_base"/>
+            <child link="cobot_base"/>
             <origin rpy="0 0 1.57080" xyz="0 0 0"/>
             <axis xyz="0 0 1"/>
         </joint>
-        <link name="head_base">
+        <link name="cobot_base">
             <visual>
                 <geometry>
@@ -22,12 +22,12 @@
             </collision>
         </link>
-        <joint name="head_joint2_to_joint1" type="revolute">
+        <joint name="cobot_joint2_to_joint1" type="revolute">
             <axis xyz="0 0 1"/>
             <limit effort = "1000.0" lower = "-2.96" upper = "2.96" velocity = "0"/>
-            <parent link="head_base"/>
-            <child link="head_link1"/>
+            <parent link="cobot_base"/>
+            <child link="cobot_link1"/>
             <origin xyz= "0 0 0.173" rpy = "0 0 0"/>
         </joint>
-        <link name="head_link1">
+        <link name="cobot_link1">
             <visual>
                 <geometry>
@@ -43,12 +43,12 @@
             </collision>
         </link>
-        <joint name="head_joint3_to_joint2" type="revolute">
+        <joint name="cobot_joint3_to_joint2" type="revolute">
             <axis xyz="0 0 1"/>
             <limit effort = "1000.0" lower = "-2.79" upper = "2.79" velocity = "0"/>
-            <parent link="head_link1"/>
-            <child link="head_link2"/>
+            <parent link="cobot_link1"/>
+            <child link="cobot_link2"/>
             <origin xyz= "-0.086 0 0" rpy = "0 1.57080 3.14"/>
         </joint>
-        <link name="head_link2">
+        <link name="cobot_link2">
             <visual>
                 <geometry>
@@ -64,12 +64,12 @@
             </collision>
         </link>
-        <joint name="head_joint4_to_joint3" type="revolute">
+        <joint name="cobot_joint4_to_joint3" type="revolute">
             <axis xyz=" 0 0 1"/>
             <limit effort = "1000.0" lower = "-2.79" upper = "2.79" velocity = "0"/>
-            <parent link="head_link2"/>
-            <child link="head_link3"/>
+            <parent link="cobot_link2"/>
+            <child link="cobot_link3"/>
             <origin xyz= "-0.13635 0 -0.086" rpy = "1.5708 0 0"/>
         </joint>
-        <link name="head_link3">
+        <link name="cobot_link3">
             <visual>
                 <geometry>
@@ -85,12 +85,12 @@
             </collision>
         </link>
-        <joint name="head_joint5_to_joint4" type="revolute">
+        <joint name="cobot_joint5_to_joint4" type="revolute">
             <axis xyz=" 0 0 1"/>
             <limit effort = "1000.0" lower = "-2.79" upper = "2.79" velocity = "0"/>
-            <parent link="head_link3"/>
-            <child link="head_link4"/>
+            <parent link="cobot_link3"/>
+            <child link="cobot_link4"/>
             <origin xyz = "-0.1195 0.082 0" rpy = " 0 0 1.57080"/>
         </joint>
-        <link name="head_link4">
+        <link name="cobot_link4">
             <visual>
                 <geometry>
@@ -106,12 +106,12 @@
             </collision>
         </link>
-        <joint name="head_joint6_to_joint5" type="revolute">
+        <joint name="cobot_joint6_to_joint5" type="revolute">
             <axis xyz="0 0 1"/>
             <limit effort = "1000.0" lower = "-2.96" upper = "2.96" velocity = "0"/>
-            <parent link="head_link4"/>
-            <child link="head_link5"/>
+            <parent link="cobot_link4"/>
+            <child link="cobot_link5"/>
             <origin xyz= "-0.09415 0 0" rpy = "0 1.5708 0"/>
         </joint>
-        <link name="head_link5">
+        <link name="cobot_link5">
             <visual>
                 <geometry>
@@ -127,12 +127,12 @@
             </collision>
         </link>
-        <joint name="head_joint6output_to_joint6" type="revolute">
+        <joint name="cobot_joint6output_to_joint6" type="revolute">
             <axis xyz="0 0 1"/>
             <limit effort = "1000.0" lower = "-3.05" upper = "3.05" velocity = "0"/>
-            <parent link="head_link5"/>
-            <child link="head_link6"/>
+            <parent link="cobot_link5"/>
+            <child link="cobot_link6"/>
             <origin xyz= "0 -0.06635 0" rpy = "1.5708 0 0"/>
         </joint>
-        <link name="head_link6">
+        <link name="cobot_link6">
             <visual>
                 <geometry>
@@ -148,4 +148,9 @@
             </collision>
         </link>
+        <joint name="cobot_joint6output_to_joint6" type="revolute">
+            <parent link="cobot_link6"/>
+            <child link="${end_link}"/>
+            <origin xyz= "0 0 0" rpy = "0 0 0"/>
+        </joint>
     </xacro:macro>
 </robot>

File: zoo/processed/Sarcomere Dynamics/Theia/xacro/theia.xacro (robot description, xacro)
@@ -42,5 +42,9 @@
     </joint>
     <link name="left_ur_base_link"/>
-	<xacro:ur5e_robot prefix="left_" base_link="left_ur_base_link" end_link="left_ee_link"/>
+    <xacro:ur5e_robot prefix="left_"
+                      base_link="left_ur_base_link"
+                      end_link="left_ee_link"
+                      joint_limits_parameters_file='joint_limits_left.yaml'
+    />
     <link name="left_ee_link"/>
     <joint name="left_gripper_fixed_joint" type="fixed">
@@ -59,5 +63,9 @@
     </joint>
     <link name="right_ur_base_link"/>
-	<xacro:ur5e_robot prefix="right_" base_link="right_ur_base_link" end_link="right_ee_link"/>
+	<xacro:ur5e_robot prefix="right_"
+                      base_link="right_ur_base_link"
+                      end_link="right_ee_link"
+                      joint_limits_parameters_file='joint_limits_right.yaml'
+    />
     <link name="right_ee_link"/>
     <joint name="right_gripper_fixed_joint" type="fixed">

Commit message: Theia updates

File: zoo/processed/Sarcomere Dynamics/Theia/xacro/artus_dex_left_macro.xacro (robot description, xacro)
@@ -242,6 +242,6 @@
 			<inertial>
 				<origin xyz="0 0 0" rpy="0 0 0"/>
-				<mass value="0" />
-				<inertia ixx="0" ixy="0"  ixz="0" iyy="0" iyz="0" izz="0" />
+				<mass value="0.025" />
+				<inertia ixx="1.666e-7" ixy="0" ixz="0" iyy="1.666e-7" iyz="0" izz="1.666e-7" />
 			</inertial>
 		</link>
@@ -264,6 +264,6 @@
 			<inertial>
 				<origin xyz="0 0 0" rpy="0 0 0"/>
-				<mass value="0" />
-				<inertia ixx="0" ixy="0"  ixz="0" iyy="0" iyz="0" izz="0" />
+				<mass value="0.025" />
+				<inertia ixx="1.666e-7" ixy="0" ixz="0" iyy="1.666e-7" iyz="0" izz="1.666e-7" />
 			</inertial>
 		</link>
@@ -286,6 +286,6 @@
 			<inertial>
 				<origin xyz="0 0 0" rpy="0 0 0"/>
-				<mass value="0" />
-				<inertia ixx="0" ixy="0"  ixz="0" iyy="0" iyz="0" izz="0" />
+				<mass value="0.025" />
+				<inertia ixx="1.666e-7" ixy="0" ixz="0" iyy="1.666e-7" iyz="0" izz="1.666e-7" />
 			</inertial>
 		</link>
@@ -308,6 +308,6 @@
 			<inertial>
 				<origin xyz="0 0 0" rpy="0 0 0"/>
-				<mass value="0" />
-				<inertia ixx="0" ixy="0"  ixz="0" iyy="0" iyz="0" izz="0" />
+				<mass value="0.025" />
+				<inertia ixx="1.666e-7" ixy="0" ixz="0" iyy="1.666e-7" iyz="0" izz="1.666e-7" />
 			</inertial>
 			<bow tags="effector"/>
@@ -363,6 +363,6 @@
 			<inertial>
 				<origin xyz="0 0 0" rpy="0 0 0"/>
-				<mass value="0" />
-				<inertia ixx="0" ixy="0"  ixz="0" iyy="0" iyz="0" izz="0" />
+				<mass value="0.025" />
+				<inertia ixx="1.666e-7" ixy="0" ixz="0" iyy="1.666e-7" iyz="0" izz="1.666e-7" />
 			</inertial>
 		</link>
@@ -385,6 +385,6 @@
 			<inertial>
 				<origin xyz="0 0 0" rpy="0 0 0"/>
-				<mass value="0" />
-				<inertia ixx="0" ixy="0"  ixz="0" iyy="0" iyz="0" izz="0" />
+				<mass value="0.025" />
+				<inertia ixx="1.666e-7" ixy="0" ixz="0" iyy="1.666e-7" iyz="0" izz="1.666e-7" />
 			</inertial>
 		</link>
@@ -407,6 +407,6 @@
 			<inertial>
 				<origin xyz="0 0 0" rpy="0 0 0"/>
-				<mass value="0" />
-				<inertia ixx="0" ixy="0"  ixz="0" iyy="0" iyz="0" izz="0" />
+				<mass value="0.025" />
+				<inertia ixx="1.666e-7" ixy="0" ixz="0" iyy="1.666e-7" iyz="0" izz="1.666e-7" />
 			</inertial>
 		</link>
@@ -429,6 +429,6 @@
 			<inertial>
 				<origin xyz="0 0 0" rpy="0 0 0"/>
-				<mass value="0" />
-				<inertia ixx="0" ixy="0"  ixz="0" iyy="0" iyz="0" izz="0" />
+				<mass value="0.025" />
+				<inertia ixx="1.666e-7" ixy="0" ixz="0" iyy="1.666e-7" iyz="0" izz="1.666e-7" />
 			</inertial>
 			<bow tags="effector"/>
@@ -484,6 +484,6 @@
 			<inertial>
 				<origin xyz="0 0 0" rpy="0 0 0"/>
-				<mass value="0" />
-				<inertia ixx="0" ixy="0"  ixz="0" iyy="0" iyz="0" izz="0" />
+				<mass value="0.025" />
+				<inertia ixx="1.666e-7" ixy="0" ixz="0" iyy="1.666e-7" iyz="0" izz="1.666e-7" />
 			</inertial>
 		</link>
@@ -506,6 +506,6 @@
 			<inertial>
 				<origin xyz="0 0 0" rpy="0 0 0"/>
-				<mass value="0" />
-				<inertia ixx="0" ixy="0"  ixz="0" iyy="0" iyz="0" izz="0" />
+				<mass value="0.025" />
+				<inertia ixx="1.666e-7" ixy="0" ixz="0" iyy="1.666e-7" iyz="0" izz="1.666e-7" />
 			</inertial>
 		</link>
@@ -528,6 +528,6 @@
 			<inertial>
 				<origin xyz="0 0 0" rpy="0 0 0"/>
-				<mass value="0" />
-				<inertia ixx="0" ixy="0"  ixz="0" iyy="0" iyz="0" izz="0" />
+				<mass value="0.025" />
+				<inertia ixx="1.666e-7" ixy="0" ixz="0" iyy="1.666e-7" iyz="0" izz="1.666e-7" />
 			</inertial>
 		</link>
@@ -550,6 +550,6 @@
 			<inertial>
 				<origin xyz="0 0 0" rpy="0 0 0"/>
-				<mass value="0" />
-				<inertia ixx="0" ixy="0"  ixz="0" iyy="0" iyz="0" izz="0" />
+				<mass value="0.025" />
+				<inertia ixx="1.666e-7" ixy="0" ixz="0" iyy="1.666e-7" iyz="0" izz="1.666e-7" />
 			</inertial>
 			<bow tags="effector"/>
@@ -605,6 +605,6 @@
 			<inertial>
 				<origin xyz="0 0 0" rpy="0 0 0"/>
-				<mass value="0" />
-				<inertia ixx="0" ixy="0"  ixz="0" iyy="0" iyz="0" izz="0" />
+				<mass value="0.025" />
+				<inertia ixx="1.666e-7" ixy="0" ixz="0" iyy="1.666e-7" iyz="0" izz="1.666e-7" />
 			</inertial>
 		</link>
@@ -627,6 +627,6 @@
 			<inertial>
 				<origin xyz="0 0 0" rpy="0 0 0"/>
-				<mass value="0" />
-				<inertia ixx="0" ixy="0"  ixz="0" iyy="0" iyz="0" izz="0" />
+				<mass value="0.025" />
+				<inertia ixx="1.666e-7" ixy="0" ixz="0" iyy="1.666e-7" iyz="0" izz="1.666e-7" />
 			</inertial>
 		</link>
@@ -649,6 +649,6 @@
 			<inertial>
 				<origin xyz="0 0 0" rpy="0 0 0"/>
-				<mass value="0" />
-				<inertia ixx="0" ixy="0"  ixz="0" iyy="0" iyz="0" izz="0" />
+				<mass value="0.025" />
+				<inertia ixx="1.666e-7" ixy="0" ixz="0" iyy="1.666e-7" iyz="0" izz="1.666e-7" />
 			</inertial>
 		</link>
@@ -671,6 +671,6 @@
 			<inertial>
 				<origin xyz="0 0 0" rpy="0 0 0"/>
-				<mass value="0" />
-				<inertia ixx="0" ixy="0"  ixz="0" iyy="0" iyz="0" izz="0" />
+				<mass value="0.025" />
+				<inertia ixx="1.666e-7" ixy="0" ixz="0" iyy="1.666e-7" iyz="0" izz="1.666e-7" />
 			</inertial>
 			<bow tags="effector"/>
@@ -726,6 +726,6 @@
 			<inertial>
 				<origin xyz="0 0 0" rpy="0 0 0"/>
-				<mass value="0" />
-				<inertia ixx="0" ixy="0"  ixz="0" iyy="0" iyz="0" izz="0" />
+				<mass value="0.025" />
+				<inertia ixx="1.666e-7" ixy="0" ixz="0" iyy="1.666e-7" iyz="0" izz="1.666e-7" />
 			</inertial>
 		</link>
@@ -748,6 +748,6 @@
 			<inertial>
 				<origin xyz="0 0 0" rpy="0 0 0"/>
-				<mass value="0" />
-				<inertia ixx="0" ixy="0"  ixz="0" iyy="0" iyz="0" izz="0" />
+				<mass value="0.025" />
+				<inertia ixx="1.666e-7" ixy="0" ixz="0" iyy="1.666e-7" iyz="0" izz="1.666e-7" />
 			</inertial>
 		</link>
@@ -770,6 +770,6 @@
 			<inertial>
 				<origin xyz="0 0 0" rpy="0 0 0"/>
-				<mass value="0" />
-				<inertia ixx="0" ixy="0"  ixz="0" iyy="0" iyz="0" izz="0" />
+				<mass value="0.025" />
+				<inertia ixx="1.666e-7" ixy="0" ixz="0" iyy="1.666e-7" iyz="0" izz="1.666e-7" />
 			</inertial>
 		</link>
@@ -792,6 +792,6 @@
 			<inertial>
 				<origin xyz="0 0 0" rpy="0 0 0"/>
-				<mass value="0" />
-				<inertia ixx="0" ixy="0"  ixz="0" iyy="0" iyz="0" izz="0" />
+				<mass value="0.025" />
+				<inertia ixx="1.666e-7" ixy="0" ixz="0" iyy="1.666e-7" iyz="0" izz="1.666e-7" />
 			</inertial>
 			<bow tags="effector"/>

File: zoo/processed/Sarcomere Dynamics/Theia/xacro/artus_dex_right_macro.xacro (robot description, xacro)
@@ -272,6 +272,6 @@
 			<inertial>
 				<origin xyz="0 0 0" rpy="0 0 0"/>
-				<mass value="0" />
-				<inertia ixx="0" ixy="0"  ixz="0" iyy="0" iyz="0" izz="0" />
+				<mass value="0.025" />
+				<inertia ixx="1.666e-7" ixy="0" ixz="0" iyy="1.666e-7" iyz="0" izz="1.666e-7" />
 			</inertial>
 		</link>
@@ -294,6 +294,6 @@
 			<inertial>
 				<origin xyz="0 0 0" rpy="0 0 0"/>
-				<mass value="0" />
-				<inertia ixx="0" ixy="0"  ixz="0" iyy="0" iyz="0" izz="0" />
+				<mass value="0.025" />
+				<inertia ixx="1.666e-7" ixy="0" ixz="0" iyy="1.666e-7" iyz="0" izz="1.666e-7" />
 			</inertial>
 		</link>
@@ -316,6 +316,6 @@
 			<inertial>
 				<origin xyz="0 0 0" rpy="0 0 0"/>
-				<mass value="0" />
-				<inertia ixx="0" ixy="0"  ixz="0" iyy="0" iyz="0" izz="0" />
+				<mass value="0.025" />
+				<inertia ixx="1.666e-7" ixy="0" ixz="0" iyy="1.666e-7" iyz="0" izz="1.666e-7" />
 			</inertial>
 		</link>
@@ -338,6 +338,6 @@
 			<inertial>
 				<origin xyz="0 0 0" rpy="0 0 0"/>
-				<mass value="0" />
-				<inertia ixx="0" ixy="0"  ixz="0" iyy="0" iyz="0" izz="0" />
+				<mass value="0.025" />
+				<inertia ixx="1.666e-7" ixy="0" ixz="0" iyy="1.666e-7" iyz="0" izz="1.666e-7" />
 			</inertial>
 			<bow tags="effector"/>
@@ -393,6 +393,6 @@
 			<inertial>
 				<origin xyz="0 0 0" rpy="0 0 0"/>
-				<mass value="0" />
-				<inertia ixx="0" ixy="0"  ixz="0" iyy="0" iyz="0" izz="0" />
+				<mass value="0.025" />
+				<inertia ixx="1.666e-7" ixy="0" ixz="0" iyy="1.666e-7" iyz="0" izz="1.666e-7" />
 			</inertial>
 		</link>
@@ -415,6 +415,6 @@
 			<inertial>
 				<origin xyz="0 0 0" rpy="0 0 0"/>
-				<mass value="0" />
-				<inertia ixx="0" ixy="0"  ixz="0" iyy="0" iyz="0" izz="0" />
+				<mass value="0.025" />
+				<inertia ixx="1.666e-7" ixy="0" ixz="0" iyy="1.666e-7" iyz="0" izz="1.666e-7" />
 			</inertial>
 		</link>
@@ -437,6 +437,6 @@
 			<inertial>
 				<origin xyz="0 0 0" rpy="0 0 0"/>
-				<mass value="0" />
-				<inertia ixx="0" ixy="0"  ixz="0" iyy="0" iyz="0" izz="0" />
+				<mass value="0.025" />
+				<inertia ixx="1.666e-7" ixy="0" ixz="0" iyy="1.666e-7" iyz="0" izz="1.666e-7" />
 			</inertial>
 		</link>
@@ -459,6 +459,6 @@
 			<inertial>
 				<origin xyz="0 0 0" rpy="0 0 0"/>
-				<mass value="0" />
-				<inertia ixx="0" ixy="0"  ixz="0" iyy="0" iyz="0" izz="0" />
+				<mass value="0.025" />
+				<inertia ixx="1.666e-7" ixy="0" ixz="0" iyy="1.666e-7" iyz="0" izz="1.666e-7" />
 			</inertial>
 			<bow tags="effector"/>
@@ -514,6 +514,6 @@
 			<inertial>
 				<origin xyz="0 0 0" rpy="0 0 0"/>
-				<mass value="0" />
-				<inertia ixx="0" ixy="0"  ixz="0" iyy="0" iyz="0" izz="0" />
+				<mass value="0.025" />
+				<inertia ixx="1.666e-7" ixy="0" ixz="0" iyy="1.666e-7" iyz="0" izz="1.666e-7" />
 			</inertial>
 		</link>
@@ -536,6 +536,6 @@
 			<inertial>
 				<origin xyz="0 0 0" rpy="0 0 0"/>
-				<mass value="0" />
-				<inertia ixx="0" ixy="0"  ixz="0" iyy="0" iyz="0" izz="0" />
+				<mass value="0.025" />
+				<inertia ixx="1.666e-7" ixy="0" ixz="0" iyy="1.666e-7" iyz="0" izz="1.666e-7" />
 			</inertial>
 		</link>
@@ -558,6 +558,6 @@
 			<inertial>
 				<origin xyz="0 0 0" rpy="0 0 0"/>
-				<mass value="0" />
-				<inertia ixx="0" ixy="0"  ixz="0" iyy="0" iyz="0" izz="0" />
+				<mass value="0.025" />
+				<inertia ixx="1.666e-7" ixy="0" ixz="0" iyy="1.666e-7" iyz="0" izz="1.666e-7" />
 			</inertial>
 		</link>
@@ -580,6 +580,6 @@
 			<inertial>
 				<origin xyz="0 0 0" rpy="0 0 0"/>
-				<mass value="0" />
-				<inertia ixx="0" ixy="0"  ixz="0" iyy="0" iyz="0" izz="0" />
+				<mass value="0.025" />
+				<inertia ixx="1.666e-7" ixy="0" ixz="0" iyy="1.666e-7" iyz="0" izz="1.666e-7" />
 			</inertial>
 			<bow tags="effector"/>
@@ -635,6 +635,6 @@
 			<inertial>
 				<origin xyz="0 0 0" rpy="0 0 0"/>
-				<mass value="0" />
-				<inertia ixx="0" ixy="0"  ixz="0" iyy="0" iyz="0" izz="0" />
+				<mass value="0.025" />
+				<inertia ixx="1.666e-7" ixy="0" ixz="0" iyy="1.666e-7" iyz="0" izz="1.666e-7" />
 			</inertial>
 		</link>
@@ -657,6 +657,6 @@
 			<inertial>
 				<origin xyz="0 0 0" rpy="0 0 0"/>
-				<mass value="0" />
-				<inertia ixx="0" ixy="0"  ixz="0" iyy="0" iyz="0" izz="0" />
+				<mass value="0.025" />
+				<inertia ixx="1.666e-7" ixy="0" ixz="0" iyy="1.666e-7" iyz="0" izz="1.666e-7" />
 			</inertial>
 		</link>
@@ -679,6 +679,6 @@
 			<inertial>
 				<origin xyz="0 0 0" rpy="0 0 0"/>
-				<mass value="0" />
-				<inertia ixx="0" ixy="0"  ixz="0" iyy="0" iyz="0" izz="0" />
+				<mass value="0.025" />
+				<inertia ixx="1.666e-7" ixy="0" ixz="0" iyy="1.666e-7" iyz="0" izz="1.666e-7" />
 			</inertial>
 		</link>
@@ -701,6 +701,6 @@
 			<inertial>
 				<origin xyz="0 0 0" rpy="0 0 0"/>
-				<mass value="0" />
-				<inertia ixx="0" ixy="0"  ixz="0" iyy="0" iyz="0" izz="0" />
+				<mass value="0.025" />
+				<inertia ixx="1.666e-7" ixy="0" ixz="0" iyy="1.666e-7" iyz="0" izz="1.666e-7" />
 			</inertial>
 			<bow tags="effector"/>
@@ -756,6 +756,6 @@
 			<inertial>
 				<origin xyz="0 0 0" rpy="0 0 0"/>
-				<mass value="0" />
-				<inertia ixx="0" ixy="0"  ixz="0" iyy="0" iyz="0" izz="0" />
+				<mass value="0.025" />
+				<inertia ixx="1.666e-7" ixy="0" ixz="0" iyy="1.666e-7" iyz="0" izz="1.666e-7" />
 			</inertial>
 		</link>
@@ -778,6 +778,6 @@
 			<inertial>
 				<origin xyz="0 0 0" rpy="0 0 0"/>
-				<mass value="0" />
-				<inertia ixx="0" ixy="0"  ixz="0" iyy="0" iyz="0" izz="0" />
+				<mass value="0.025" />
+				<inertia ixx="1.666e-7" ixy="0" ixz="0" iyy="1.666e-7" iyz="0" izz="1.666e-7" />
 			</inertial>
 		</link>
@@ -800,6 +800,6 @@
 			<inertial>
 				<origin xyz="0 0 0" rpy="0 0 0"/>
-				<mass value="0" />
-				<inertia ixx="0" ixy="0"  ixz="0" iyy="0" iyz="0" izz="0" />
+				<mass value="0.025" />
+				<inertia ixx="1.666e-7" ixy="0" ixz="0" iyy="1.666e-7" iyz="0" izz="1.666e-7" />
 			</inertial>
 		</link>
@@ -822,6 +822,6 @@
 			<inertial>
 				<origin xyz="0 0 0" rpy="0 0 0"/>
-				<mass value="0" />
-				<inertia ixx="0" ixy="0"  ixz="0" iyy="0" iyz="0" izz="0" />
+				<mass value="0.025" />
+				<inertia ixx="1.666e-7" ixy="0" ixz="0" iyy="1.666e-7" iyz="0" izz="1.666e-7" />
 			</inertial>
 			<bow tags="effector"/>

File: zoo/processed/Sarcomere Dynamics/Theia/xacro/theia.xacro (robot description, xacro)
@@ -9,9 +9,10 @@
         <parent link="base_link"/>
         <child link="table"/>
-        <origin rpy="0 0 0" xyz="0.2 0 -0.4"/>
+        <origin rpy="0 0 0" xyz="0 0 0"/>
         <axis xyz="0 0 1"/>
     </joint>
     <link name="table">
         <visual>
+            <origin rpy="0.0 0.0 0.0" xyz="0.2 0.0 -0.4"/>
             <geometry>
                 <box size="0.6 1.2 0.8"/>
@@ -19,4 +20,5 @@
         </visual>
         <collision>
+            <origin rpy="0.0 0.0 0.0" xyz="0.2 0.0 -0.4"/>
             <geometry>
                 <box size="0.6 1.2 0.8"/>
@@ -32,5 +34,5 @@
         <parent link="table"/>
         <child link="head_base_link"/>
-        <origin xyz="0 0 0" rpy="0 0 -1.5708"/>
+        <origin xyz="-0.05 0 0" rpy="0 0 -1.5708"/>
     </joint>
     <link name="head_base_link">
@@ -44,5 +46,5 @@
       <parent link="table" />
       <child link="left_ur_base_link" />
-      <origin xyz="0 0.4 0" rpy="0 0 0" />
+      <origin xyz="0.1 0.4 0" rpy="0 0 0" />
     </joint>
     <link name="left_ur_base_link"/>
@@ -65,5 +67,5 @@
       <parent link="table" />
       <child link="right_ur_base_link" />
-      <origin xyz="0 -0.4 0" rpy="0 0 3.148"/>
+      <origin xyz="0.1 -0.4 0" rpy="0 0 3.148"/>
     </joint>
     <link name="right_ur_base_link"/>
