Commit message: Sarcomere Theia update

File: zoo/processed/Sarcomere Dynamics/Theia/xacro/artus_dex_right_macro.xacro (robot description, xacro)
@@ -341,4 +341,5 @@
 				<inertia ixx="0" ixy="0"  ixz="0" iyy="0" iyz="0" izz="0" />
 			</inertial>
+			<bow tags="effector"/>
 		</link>
 		<joint name="Rpinky_34" type="revolute">
@@ -461,4 +462,5 @@
 				<inertia ixx="0" ixy="0"  ixz="0" iyy="0" iyz="0" izz="0" />
 			</inertial>
+			<bow tags="effector"/>
 		</link>
 		<joint name="Rring_34" type="revolute">
@@ -581,4 +583,5 @@
 				<inertia ixx="0" ixy="0"  ixz="0" iyy="0" iyz="0" izz="0" />
 			</inertial>
+			<bow tags="effector"/>
 		</link>
 		<joint name="Rmiddle_34" type="revolute">
@@ -701,4 +704,5 @@
 				<inertia ixx="0" ixy="0"  ixz="0" iyy="0" iyz="0" izz="0" />
 			</inertial>
+			<bow tags="effector"/>
 		</link>
 		<joint name="Rindex_34" type="revolute">
@@ -817,8 +821,9 @@
 			</collision>
 			<inertial>
-			<origin xyz="0 0 0" rpy="0 0 0"/>
-			<mass value="0" />
-			<inertia ixx="0" ixy="0"  ixz="0" iyy="0" iyz="0" izz="0" />
-			</inertial>
+				<origin xyz="0 0 0" rpy="0 0 0"/>
+				<mass value="0" />
+				<inertia ixx="0" ixy="0"  ixz="0" iyy="0" iyz="0" izz="0" />
+			</inertial>
+			<bow tags="effector"/>
 		</link>
 		<joint name="Rthumb_34" type="revolute">

File: zoo/processed/Sarcomere Dynamics/Theia/xacro/theia.xacro (robot description, xacro)
@@ -34,6 +34,11 @@
         <origin xyz="0 0 0" rpy="0 0 -1.5708"/>
     </joint>
-    <link name="head_base_link"/>
-    <xacro:elephantbot_mycobot_pro_320 base_link="head_base_link"/>
+    <link name="head_base_link">
+        <bow tags="limb"/>
+    </link>
+    <xacro:elephantbot_mycobot_pro_320 base_link="head_base_link" end_link="head_end_link"/>
+    <link name="head_end_link">
+        <bow tags="gripper"/>
+    </link>
 	<joint name="left_ur_fixed_joint" type="fixed">
       <parent link="base_link" />

Commit message: Xacro prefix fixes

File: zoo/processed/Sarcomere Dynamics/Theia/xacro/artus_dex_right_macro.xacro (robot description, xacro)
@@ -2,5 +2,5 @@
 <robot xmlns:xacro="http://ros.org/wiki/xacro">
 	<xacro:macro name="artus_dex_right" params="prefix base_link mesh_dir">
-		<joint name="virtual" type="fixed">
+		<joint name="${prefix}virtual" type="fixed">
 			<origin xyz="0 0 0" rpy="0 0 0"/>
 			<parent link="${base_link}"/>
@@ -254,5 +254,5 @@
 			</inertial>
 		</link>
-		<link name="part_1_1">
+		<link name="${prefix}part_1_1">
 			<visual>
 				<origin xyz="-0.0049999999999999766853 0 -0.018500000000000103167" rpy="0 0 0" />
