Commit message: Theia xacro updates

File: zoo/processed/Sarcomere Dynamics/Theia/xacro/elephantbot_mycobot320_macro.xacro (robot description, xacro)
@@ -148,5 +148,5 @@
             </collision>
         </link>
-        <joint name="cobot_joint6output_to_joint6" type="revolute">
+        <joint name="tool_joint" type="revolute">
             <parent link="cobot_link6"/>
             <child link="${end_link}"/>

File: zoo/processed/Sarcomere Dynamics/Theia/xacro/theia.xacro (robot description, xacro)
@@ -30,5 +30,5 @@
     </link>
     <joint name="head_fixed_joint" type="fixed">
-        <parent link="base_link"/>
+        <parent link="table"/>
         <child link="head_base_link"/>
         <origin xyz="0 0 0" rpy="0 0 -1.5708"/>
@@ -42,5 +42,5 @@
     </link>
 	<joint name="left_ur_fixed_joint" type="fixed">
-      <parent link="base_link" />
+      <parent link="table" />
       <child link="left_ur_base_link" />
       <origin xyz="0 0.4 0" rpy="0 0 0" />
@@ -63,5 +63,5 @@
     <xacro:artus_dex_left base_link="left_gripper_base" mesh_dir="left_artus"/>
 	<joint name="right_ur_fixed_joint" type="fixed">
-      <parent link="base_link" />
+      <parent link="table" />
       <child link="right_ur_base_link" />
       <origin xyz="0 -0.4 0" rpy="0 0 3.148"/>

Commit message: Elephant bot update

File: zoo/processed/Sarcomere Dynamics/Theia/xacro/elephantbot_mycobot320_macro.xacro (robot description, xacro)
@@ -11,5 +11,5 @@
             <visual>
                 <geometry>
-                    <mesh filename="meshes/elephantbot/base.dae"/>
+                    <mesh filename="meshes/elephantbot/base.dae" scale="0.001 0.001 0.001"/>
                 </geometry>
                 <origin xyz = "0.0 0 0 " rpy = "0 0 1.5708"/>
@@ -17,5 +17,5 @@
             <collision>
                 <geometry>
-                    <mesh filename="meshes/elephantbot/base.dae"/>
+                    <mesh filename="meshes/elephantbot/base.dae" scale="0.001 0.001 0.001"/>
                 </geometry>
                 <origin xyz = "0.0 0 0 " rpy = "0 0 1.5708"/>
@@ -32,5 +32,5 @@
             <visual>
                 <geometry>
-                    <mesh filename="meshes/elephantbot/link1.dae"/>
+                    <mesh filename="meshes/elephantbot/link1.dae" scale="0.001 0.001 0.001"/>
                 </geometry>
                 <origin xyz = "0.0 0.0 -0.078 " rpy = " 0 0 1.5708"/>
@@ -38,5 +38,5 @@
             <collision>
                 <geometry>
-                    <mesh filename="meshes/elephantbot/link1.dae"/>
+                    <mesh filename="meshes/elephantbot/link1.dae" scale="0.001 0.001 0.001"/>
                 </geometry>
                 <origin xyz = "0.0 0.0 -0.078 " rpy = " 0 0 1.5708"/>
@@ -53,5 +53,5 @@
             <visual>
                 <geometry>
-                    <mesh filename="meshes/elephantbot/link2.dae"/>
+                    <mesh filename="meshes/elephantbot/link2.dae" scale="0.001 0.001 0.001"/>
                 </geometry>
                 <origin xyz = "0.0 0.0 -0.04" rpy = " 1.5708 3.14 0"/>
@@ -59,5 +59,5 @@
             <collision>
                 <geometry>
-                    <mesh filename="meshes/elephantbot/link2.dae"/>
+                    <mesh filename="meshes/elephantbot/link2.dae" scale="0.001 0.001 0.001"/>
                 </geometry>
                 <origin xyz = "0.0 0.0 -0.04" rpy = " 1.5708 3.14 0"/>
@@ -74,5 +74,5 @@
             <visual>
                 <geometry>
-                    <mesh filename="meshes/elephantbot/link3.dae"/>
+                    <mesh filename="meshes/elephantbot/link3.dae" scale="0.001 0.001 0.001"/>
                 </geometry>
                 <origin xyz = "0.0 0.04 0 " rpy = "1.5708 0 -1.5708"/>
@@ -80,5 +80,5 @@
             <collision>
                 <geometry>
-                    <mesh filename="meshes/elephantbot/link3.dae"/>
+                    <mesh filename="meshes/elephantbot/link3.dae" scale="0.001 0.001 0.001"/>
                 </geometry>
                 <origin xyz = "0.0 0.04 0 " rpy = "1.5708 0 -1.5708"/>
@@ -95,5 +95,5 @@
             <visual>
                 <geometry>
-                    <mesh filename="meshes/elephantbot/link4.dae"/>
+                    <mesh filename="meshes/elephantbot/link4.dae" scale="0.001 0.001 0.001"/>
                 </geometry>
                 <origin xyz = "-0.0024 -0.05 0" rpy = "1.5708 0 -1.5708"/>
@@ -101,5 +101,5 @@
             <collision>
                 <geometry>
-                    <mesh filename="meshes/elephantbot/link4.dae"/>
+                    <mesh filename="meshes/elephantbot/link4.dae" scale="0.001 0.001 0.001"/>
                 </geometry>
                 <origin xyz = "-0.0024 -0.05 0" rpy = "1.5708 0 -1.5708"/>
@@ -116,5 +116,5 @@
             <visual>
                 <geometry>
-                    <mesh filename="meshes/elephantbot/link5.dae"/>
+                    <mesh filename="meshes/elephantbot/link5.dae" scale="0.001 0.001 0.001"/>
                 </geometry>
                 <origin xyz = "0.0 -0.0015 0.05" rpy = "3.14 0 1.5708"/>
@@ -122,5 +122,5 @@
             <collision>
                 <geometry>
-                    <mesh filename="meshes/elephantbot/link5.dae"/>
+                    <mesh filename="meshes/elephantbot/link5.dae" scale="0.001 0.001 0.001"/>
                 </geometry>
                 <origin xyz = "0.0 -0.0015 0.05" rpy = "3.14 0 1.5708"/>
@@ -137,5 +137,5 @@
             <visual>
                 <geometry>
-                    <mesh filename="meshes/elephantbot/link6.dae"/>
+                    <mesh filename="meshes/elephantbot/link6.dae" scale="0.001 0.001 0.001"/>
                 </geometry>
                 <origin xyz = "0.0 0.0 -0.0215 " rpy = " 1.5708 1.5708 0"/>
@@ -143,5 +143,5 @@
             <collision>
                 <geometry>
-                    <mesh filename="meshes/elephantbot/link6.dae"/>
+                    <mesh filename="meshes/elephantbot/link6.dae" scale="0.001 0.001 0.001"/>
                 </geometry>
                 <origin xyz = "0.0 0.0 -0.0215 " rpy = " 1.5708 1.5708 0"/>

Commit message: Elephantbot fixed

File: zoo/processed/Sarcomere Dynamics/Theia/xacro/elephantbot_mycobot320_macro.xacro (robot description, xacro)
@@ -13,5 +13,5 @@
                     <mesh filename="meshes/elephantbot/base.dae" scale="0.001 0.001 0.001"/>
                 </geometry>
-                <origin xyz = "0.0 0 0 " rpy = "0 0 1.5708"/>
+                <origin xyz="0.0 0 0 " rpy="0 0 1.5708"/>
             </visual>
             <collision>
@@ -19,13 +19,13 @@
                     <mesh filename="meshes/elephantbot/base.dae" scale="0.001 0.001 0.001"/>
                 </geometry>
-                <origin xyz = "0.0 0 0 " rpy = "0 0 1.5708"/>
+                <origin xyz="0.0 0 0" rpy="0 0 1.5708"/>
             </collision>
         </link>
         <joint name="cobot_joint2_to_joint1" type="revolute">
             <axis xyz="0 0 1"/>
-            <limit effort = "1000.0" lower = "-2.96" upper = "2.96" velocity = "0"/>
+            <limit effort="1000.0" lower="-2.96" upper="2.96" velocity="0"/>
             <parent link="cobot_base"/>
             <child link="cobot_link1"/>
-            <origin xyz= "0 0 0.173" rpy = "0 0 0"/>
+            <origin xyz="0 0 0.173" rpy="0 0 0"/>
         </joint>
         <link name="cobot_link1">
@@ -34,5 +34,5 @@
                     <mesh filename="meshes/elephantbot/link1.dae" scale="0.001 0.001 0.001"/>
                 </geometry>
-                <origin xyz = "0.0 0.0 -0.078 " rpy = " 0 0 1.5708"/>
+                <origin xyz="0.0 0.0 -0.078" rpy="0 0 0"/>
             </visual>
             <collision>
@@ -40,13 +40,13 @@
                     <mesh filename="meshes/elephantbot/link1.dae" scale="0.001 0.001 0.001"/>
                 </geometry>
-                <origin xyz = "0.0 0.0 -0.078 " rpy = " 0 0 1.5708"/>
+                <origin xyz="0.0 0.0 -0.078 " rpy="0 0 0"/>
             </collision>
         </link>
         <joint name="cobot_joint3_to_joint2" type="revolute">
             <axis xyz="0 0 1"/>
-            <limit effort = "1000.0" lower = "-2.79" upper = "2.79" velocity = "0"/>
+            <limit effort="1000.0" lower="-2.79" upper="2.79" velocity="0"/>
             <parent link="cobot_link1"/>
             <child link="cobot_link2"/>
-            <origin xyz= "-0.086 0 0" rpy = "0 1.57080 3.14"/>
+            <origin xyz="-0.086 0 0" rpy="0 1.57080 3.14"/>
         </joint>
         <link name="cobot_link2">
@@ -55,5 +55,5 @@
                     <mesh filename="meshes/elephantbot/link2.dae" scale="0.001 0.001 0.001"/>
                 </geometry>
-                <origin xyz = "0.0 0.0 -0.04" rpy = " 1.5708 3.14 0"/>
+                <origin xyz="0.0 0.0 -0.04" rpy="3.1416 1.5708 0"/>
             </visual>
             <collision>
@@ -61,13 +61,13 @@
                     <mesh filename="meshes/elephantbot/link2.dae" scale="0.001 0.001 0.001"/>
                 </geometry>
-                <origin xyz = "0.0 0.0 -0.04" rpy = " 1.5708 3.14 0"/>
+                <origin xyz="0.0 0.0 -0.04" rpy="3.1416 1.5708 0"/>
             </collision>
         </link>
         <joint name="cobot_joint4_to_joint3" type="revolute">
-            <axis xyz=" 0 0 1"/>
-            <limit effort = "1000.0" lower = "-2.79" upper = "2.79" velocity = "0"/>
+            <axis xyz="0 0 1"/>
+            <limit effort="1000.0" lower="-2.79" upper="2.79" velocity="0"/>
             <parent link="cobot_link2"/>
             <child link="cobot_link3"/>
-            <origin xyz= "-0.13635 0 -0.086" rpy = "1.5708 0 0"/>
+            <origin xyz="-0.13635 0 -0.086" rpy="0 0 0"/>
         </joint>
         <link name="cobot_link3">
@@ -76,5 +76,5 @@
                     <mesh filename="meshes/elephantbot/link3.dae" scale="0.001 0.001 0.001"/>
                 </geometry>
-                <origin xyz = "0.0 0.04 0 " rpy = "1.5708 0 -1.5708"/>
+                <origin xyz="0.0 0.0 0.04" rpy="1.5708 1.5708 -1.5708"/>
             </visual>
             <collision>
@@ -82,13 +82,13 @@
                     <mesh filename="meshes/elephantbot/link3.dae" scale="0.001 0.001 0.001"/>
                 </geometry>
-                <origin xyz = "0.0 0.04 0 " rpy = "1.5708 0 -1.5708"/>
+                <origin xyz="0.0 0.0 0.04" rpy="1.5708 1.5708 -1.5708"/>
             </collision>
         </link>
         <joint name="cobot_joint5_to_joint4" type="revolute">
-            <axis xyz=" 0 0 1"/>
-            <limit effort = "1000.0" lower = "-2.79" upper = "2.79" velocity = "0"/>
+            <axis xyz="0 0 1"/>
+            <limit effort="1000.0" lower="-2.79" upper="2.79" velocity="0"/>
             <parent link="cobot_link3"/>
             <child link="cobot_link4"/>
-            <origin xyz = "-0.1195 0.082 0" rpy = " 0 0 1.57080"/>
+            <origin xyz="-0.1195 0 0.082" rpy="0 0 1.57080"/>
         </joint>
         <link name="cobot_link4">
@@ -97,5 +97,5 @@
                     <mesh filename="meshes/elephantbot/link4.dae" scale="0.001 0.001 0.001"/>
                 </geometry>
-                <origin xyz = "-0.0024 -0.05 0" rpy = "1.5708 0 -1.5708"/>
+                <origin xyz="0 0.0029 -0.05" rpy="-1.5708 1.5708 0"/>
             </visual>
             <collision>
@@ -103,13 +103,13 @@
                     <mesh filename="meshes/elephantbot/link4.dae" scale="0.001 0.001 0.001"/>
                 </geometry>
-                <origin xyz = "-0.0024 -0.05 0" rpy = "1.5708 0 -1.5708"/>
+                <origin xyz="0 0.0029 -0.05" rpy="-1.5708 1.5708 0"/>
             </collision>
         </link>
         <joint name="cobot_joint6_to_joint5" type="revolute">
-            <axis xyz="0 0 1"/>
-            <limit effort = "1000.0" lower = "-2.96" upper = "2.96" velocity = "0"/>
+            <axis xyz="0 1 0"/>
+            <limit effort="1000.0" lower="-2.96" upper="2.96" velocity="0"/>
             <parent link="cobot_link4"/>
             <child link="cobot_link5"/>
-            <origin xyz= "-0.09415 0 0" rpy = "0 1.5708 0"/>
+            <origin xyz="0 0.09415 0" rpy="0 1.5708 0"/>
         </joint>
         <link name="cobot_link5">
@@ -118,5 +118,5 @@
                     <mesh filename="meshes/elephantbot/link5.dae" scale="0.001 0.001 0.001"/>
                 </geometry>
-                <origin xyz = "0.0 -0.0015 0.05" rpy = "3.14 0 1.5708"/>
+                <origin xyz="0.0015 -0.05 0" rpy="-1.5708 0 0"/>
             </visual>
             <collision>
@@ -124,13 +124,13 @@
                     <mesh filename="meshes/elephantbot/link5.dae" scale="0.001 0.001 0.001"/>
                 </geometry>
-                <origin xyz = "0.0 -0.0015 0.05" rpy = "3.14 0 1.5708"/>
+                <origin xyz="0.0015 -0.05 0" rpy="-1.5708 0 0"/>
             </collision>
         </link>
         <joint name="cobot_joint6output_to_joint6" type="revolute">
-            <axis xyz="0 0 1"/>
-            <limit effort = "1000.0" lower = "-3.05" upper = "3.05" velocity = "0"/>
+            <axis xyz="1 0 0"/>
+            <limit effort="1000.0" lower="-3.05" upper="3.05" velocity="0"/>
             <parent link="cobot_link5"/>
             <child link="cobot_link6"/>
-            <origin xyz= "0 -0.06635 0" rpy = "1.5708 0 0"/>
+            <origin xyz="-0.06635 0 0" rpy="1.5708 0 0"/>
         </joint>
         <link name="cobot_link6">
@@ -139,5 +139,5 @@
                     <mesh filename="meshes/elephantbot/link6.dae" scale="0.001 0.001 0.001"/>
                 </geometry>
-                <origin xyz = "0.0 0.0 -0.0215 " rpy = " 1.5708 1.5708 0"/>
+                <origin xyz="0.0215 0.0 0.0" rpy="3.14 0 0"/>
             </visual>
             <collision>
@@ -145,5 +145,5 @@
                     <mesh filename="meshes/elephantbot/link6.dae" scale="0.001 0.001 0.001"/>
                 </geometry>
-                <origin xyz = "0.0 0.0 -0.0215 " rpy = " 1.5708 1.5708 0"/>
+                <origin xyz="0.0215 0.0 0.0" rpy="3.14 0 0"/>
             </collision>
         </link>
@@ -151,5 +151,5 @@
             <parent link="cobot_link6"/>
             <child link="${end_link}"/>
-            <origin xyz= "0 0 0" rpy = "0 0 0"/>
+            <origin xyz="0 0 0" rpy="0 0 0"/>
         </joint>
     </xacro:macro>
