Commit message: Addition of camera to Theia

File: zoo/processed/Sarcomere Dynamics/Theia/xacro/theia.xacro (robot description, xacro)
@@ -43,4 +43,11 @@
         <bow tags="gripper"/>
     </link>
+    <joint name="HeadCamera_fixed_joint" type="fixed">
+        <parent link="head_end_link"/>
+        <child link="FrontCamera_frame"/>
+        <origin rpy="0 0 0" xyz="0.28 0 0"/>
+        <axis xyz="0 0 0"/>
+    </joint>
+    <link name="FrontCamera_frame"/>
 	<joint name="left_ur_fixed_joint" type="fixed">
       <parent link="table" />
@@ -85,3 +92,25 @@
     </link>
     <xacro:artus_dex_right base_link="right_gripper_base" mesh_dir="right_artus"/>
+    <gazebo reference="HeadCamera_frame">
+        <sensor name="HeadCamera" type="camera">
+          <update_rate>5.0</update_rate>
+          <camera name="head_camera">
+            <horizontal_fov>1.06290551</horizontal_fov>
+            <image>
+              <width>640</width>
+              <height>480</height>
+              <format>R8G8B8</format>
+            </image>
+            <clip>
+              <near>0.3</near>
+              <far>500</far>
+            </clip>
+            <noise>
+              <type>gaussian</type>
+              <mean>0.0</mean>
+              <stddev>0.007</stddev>
+            </noise>
+          </camera>
+        </sensor>
+    </gazebo>
 </robot>

Commit message: Added missing bow tags

File: zoo/processed/Sarcomere Dynamics/Theia/xacro/theia.xacro (robot description, xacro)
@@ -55,5 +55,7 @@
       <origin xyz="0.1 0.4 0" rpy="0 0 0" />
     </joint>
-    <link name="left_ur_base_link"/>
+    <link name="left_ur_base_link">
+        <bow tags="limb"/>
+    </link>
     <xacro:ur5e_robot prefix="left_"
                       base_link="left_ur_base_link"
@@ -76,5 +78,7 @@
       <origin xyz="0.1 -0.4 0" rpy="0 0 3.148"/>
     </joint>
-    <link name="right_ur_base_link"/>
+    <link name="right_ur_base_link">
+        <bow tags="limb"/>
+    </link>
 	<xacro:ur5e_robot prefix="right_"
                       base_link="right_ur_base_link"

Commit message: Theia update to tagged link

File: zoo/processed/Sarcomere Dynamics/Theia/xacro/theia.xacro (robot description, xacro)
@@ -40,14 +40,14 @@
     </link>
     <xacro:elephantbot_mycobot_pro_320 base_link="head_base_link" end_link="head_end_link"/>
-    <link name="head_end_link">
-        <bow tags="gripper"/>
-    </link>
+    <link name="head_end_link"/>
     <joint name="HeadCamera_fixed_joint" type="fixed">
         <parent link="head_end_link"/>
         <child link="FrontCamera_frame"/>
-        <origin rpy="0 0 0" xyz="0.28 0 0"/>
+        <origin rpy="0 0 0" xyz="0 0 0"/>
         <axis xyz="0 0 0"/>
     </joint>
-    <link name="FrontCamera_frame"/>
+    <link name="FrontCamera_frame">
+        <bow tags="effector"/>
+    </link>
 	<joint name="left_ur_fixed_joint" type="fixed">
       <parent link="table" />
