Commit message: tags for tiago

File: zoo/processed/PAL Robotics/Tiago/xacro/tiago.xacro (robot description, xacro)
@@ -13,5 +13,5 @@
  -->
 <robot  xmlns:xacro="http://ros.org/wiki/xacro"
-        name="tiago" >
+        name="tiago" locomotion="differential">
     <xacro:arg name="arm" default="right-arm"/> <!-- right-arm, no-arm -->
     <xacro:arg name="wrist_model" default="wrist-2010"/>

File: zoo/processed/PAL Robotics/Tiago/xacro/wheels/wheel.urdf.xacro (robot description, xacro)
@@ -14,6 +14,6 @@
 <robot xmlns:xacro="http://ros.org/wiki/xacro">
   <xacro:include filename="$(find pmb2_description)/urdf/wheels/wheel.gazebo.xacro"/>
-  <xacro:macro name="wheel" contact="wheel" params="side reflect radius width torque velocity separation parent">
-    <link name="wheel_${side}_link">
+  <xacro:macro name="wheel" params="side reflect radius width torque velocity separation parent">
+    <link name="wheel_${side}_link" contact="wheel ${radius}">
       <inertial>
         <origin xyz="0 0 ${-0.00207 * reflect}" rpy="0 0 0"/>
