Commit message: Tagged tiagos caster wheels as passive

File: zoo/processed/PAL Robotics/Tiago/xacro/wheels/caster.urdf.xacro (robot description, xacro)
@@ -15,5 +15,5 @@
   <xacro:include filename="$(find pmb2_description)/urdf/wheels/caster.gazebo.xacro"/>
   <xacro:macro name="caster" params="side radius width separation_x separation_y offset_x offset_y offset_z parent">
-    <link name="caster_${side}_1_link">
+    <link name="caster_${side}_1_link" contact="passive">
       <inertial>
         <origin xyz="-0.00634599 0.00005347 -0.02037519" rpy="0 0 0"/>
@@ -37,5 +37,5 @@
       </collision-->
     </link>
-    <link name="caster_${side}_2_link">
+    <link name="caster_${side}_2_link" contact="passive">
       <inertial>
         <origin xyz="0 0 0" rpy="0 0 0"/>
